File: PCB/ADC/ADC_MOD.kicad_sch (KiCad schematic)
At the start: 12 parts, among them J1 Conn_01x08, J2 Conn_01x02, U1 LTC2311

Commit message: ADC stuff
Parts:
- removed J1: Conn_01x08, Connector_PinHeader_2.54mm:PinHeader_1x08_P2.54mm_Vertical, symbol Connector_Generic:Conn_01x08
- added C10: 1uF, Capacitor_SMD:C_0805_2012Metric_Pad1.18x1.45mm_HandSolder, symbol Device:C_Small
- added C11, C12: 10uF, Capacitor_SMD:C_1206_3216Metric_Pad1.33x1.80mm_HandSolder, symbol Device:C_Small
- added C13, C19: C_Small, symbol Device:C_Small
- added C14, C15, C17, C21: 100nF, symbol Device:C_Small
- added C16, C20: 10uF, symbol Device:C_Small
- added C18: 220uF, symbol Device:C_Polarized_Small
- added C8: 100uF, Capacitor_THT:CP_Radial_D6.3mm_P2.50mm, symbol Device:C_Polarized_Small
- added C9: 100nF, Capacitor_SMD:C_0805_2012Metric_Pad1.18x1.45mm_HandSolder, symbol Device:C_Small
- added J1: Conn_01x02, Connector_PinHeader_2.54mm:PinHeader_1x02_P2.54mm_Vertical, symbol Connector_Generic:Conn_01x02
- added L1, L2, L3, L4: L_Small, symbol Device:L_Small
- added R3, R4: 24R9, Resistor_SMD:R_0805_2012Metric_Pad1.20x1.40mm_HandSolder, symbol Device:R_Small
- added U2: LTC2311, Package_SO:MSOP-16-1EP_3x4mm_P0.5mm_EP1.65x2.85mm_ThermalVias, symbol JRIX ADC:LTC2311-16
- added U3: REF02Z, Package_DIP:DIP-8_W7.62mm, symbol Reference_Voltage:REF02Z
- added U4: LD1117S25-TR, symbol JRIX Linear Regulator:LD1117S25
- added U5: LD1117S50-TR, symbol JRIX Linear Regulator:LD1117S50
- C5: value 10uF -> 33pF; footprint Capacitor_SMD:C_1206_3216Metric_Pad1.33x1.80mm_HandSolder -> Capacitor_SMD:C_0805_2012Metric_Pad1.18x1.45mm_HandSolder
Connections:
- net at C3.2, U1.12 (OVDD): now also C11.2, C17.1, U2.12 (OVDD), U4.2 (VOUT)
- net DAC1DO: now reaches U1.14 (SDO+)
- net DAC1DO: now also U2.14 (SDO+)
- net DAC1SCK: now reaches U1.16 (SCK+)
- net DAC1SCK: now also U2.16 (SCK+)
- net at C5.2: now also R4.2, U2.7 (AIN-); no longer U1.2 (REFIN)
- net VDD: now reaches C2.2, C7.1, U1.4 (VDD)
- net VDD: now also C6.1, C10.2, C21.1, C8.1, C9.1, U2.4 (VDD), U5.2 (VOUT); no longer C6.2
- net ~{CNV}: now reaches U1.9 (~{CNV})
- net ~{CNV}: now also U2.9 (~{CNV})
- net GND renamed GNDA
- net GNDA: now also C6.2, U1.2 (REFIN), C10.1, C11.1, C12.2, C13.2, C14.2, C15.2, C18.2, C20.2, C21.2, C8.2, C9.2, U2.1 (GND), U2.10 (~{CMOS}/LVDS), U2.11 (GND), U2.17 (GND), U2.2 (REFIN), U2.5 (GND), U2.8 (GND), U3.4 (GND), U5.1 (ADJ/GND); no longer C5.1, C6.1
- new net: C16.1, L1.1, U4.3 (VIN)
- new net: C15.1, C18.1, C20.1, L3.1, U3.2 (VIN), U5.3 (VIN)
- new net: J1.1 (Pin_1), R4.1
- new net: J1.2 (Pin_2), R3.1
- new net: C5.1, R3.2, U2.6 (AIN+)
- new net: C13.1, L2.1, L3.2
- new net: C19.1, L1.2, L4.1
- new net: C14.1, U3.6 (VOUT)
- new net: C12.1, U2.3 (REFOUT)
- new net +12V: L2.2, L4.2
- new net GNDD: C16.2, C17.2, C19.2, U4.1 (ADJ/GND)
Other:
- note added: "Keep GNDD separated from GNDA Join GNDD and GNDA in star connection away from ADCs"
- moved on the sheet: C1, C2, C3, C4, C6, C7, J2, R1, R2, U1
