File: PCB/ImpedanceAnalyzer/ANFE.kicad_sch (KiCad schematic)
At the start: 60 parts, among them U1 LTC2311, U10 OPA350, U11 OPA350, U2 LTC2311, U3 REF02Z, U4 LD1117S25-TR, U5 LD1117S50-TR, U7 LT1819, U9 OPA350

Commit message: stuff
Parts:
- added R15: R_Small, symbol Device:R_Small
Connections:
- net at C32.1, R10.2, R12.2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: now also R15.1
Changed lines of the file:
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@@
 	)
 	(junction
+		(at 137.16 74.93)
+		(diameter 0)
+		(color 0 0 0 0)
+	)
+	(junction
 		(at 297.18 115.57)
 		(diameter 0)
@@
 	(wire
 		(pts
+			(xy 137.16 74.93) (xy 137.16 85.09)
+		)
+		(stroke
+			(width 0)
+			(type default)
+		)
+	)
+	(wire
+		(pts
 			(xy 172.72 33.02) (xy 172.72 41.91)
 		)
@@
 	(wire
 		(pts
+			(xy 115.57 74.93) (xy 137.16 74.93)
+		)
+		(stroke
+			(width 0)
+			(type default)
+		)
+	)
+	(wire
+		(pts
 			(xy 245.11 82.55) (xy 245.11 83.82)
 		)
@@
 	(wire
 		(pts
+			(xy 115.57 78.74) (xy 115.57 74.93)
+		)
+		(stroke
+			(width 0)
+			(type default)
+		)
+	)
+	(wire
+		(pts
 			(xy 205.74 52.07) (xy 205.74 49.53)
 		)
@@
 	(wire
 		(pts
-			(xy 137.16 44.45) (xy 137.16 85.09)
+			(xy 137.16 44.45) (xy 137.16 74.93)
 		)
 		(stroke
@@
 					(unit 1)
 				)
+			)
+		)
+	)
+	(symbol
+		(lib_id "Device:R_Small")
+		(at 115.57 81.28 0)
+		(unit 1)
+		(exclude_from_sim no)
+		(in_bom yes)
+		(on_board yes)
+		(dnp no)
+		(fields_autoplaced yes)
+		(property "Reference" "R15"
+			(at 118.11 80.0099 0)
+			(effects
+				(font
+					(size 1.27 1.27)
+				)
+				(justify left)
+			)
+		)
+		(property "Value" "R_Small"
+			(at 118.11 82.5499 0)
+			(effects
+				(font
+					(size 1.27 1.27)
+				)
+				(justify left)
+			)
+		)
+		(property "Footprint" ""
+			(at 115.57 81.28 0)
+			(effects
+				(font
+					(size 1.27 1.27)
+				)
+				(hide yes)
+			)
+		)
+		(property "Datasheet" "~"
+			(at 115.57 81.28 0)
+			(effects
+				(font
+					(size 1.27 1.27)
+				)
+				(hide yes)
+			)
+		)
+		(property "Description" "Resistor, small symbol"
+			(at 115.57 81.28 0)
+			(effects
+				(font
+					(size 1.27 1.27)
+				)
+				(hide yes)
+			)
+		)
+		(pin "2"
+		)
+		(pin "1"
+		)
+		(instances
+			(project ""
+				(path "/08568624-f051-402a-adf3-1b03c2a769ee/7040a4f2-9510-49f8-bf95-e9f218eebebf"
+					(reference "R15")
+					(unit 1)
+				)
