File: PCB/ImpedanceAnalyzer/ANFE.kicad_sch (KiCad schematic)
At the start: 61 parts, among them U1 LTC2311, U10 OPA350, U11 OPA350, U2 LTC2311, U3 REF02Z, U4 LD1117S25-TR, U5 LD1117S50-TR, U7 LT1819, U9 OPA350

Commit message: filter work
Parts:
- removed C28: 100n, symbol Device:C_Small
- removed C29: 100u, symbol Device:C_Polarized_Small
- removed C32, C33: 2p2, symbol Device:C_Small
- removed R15: R_Small, symbol Device:R_Small
- removed unit 2 of U10
- removed unit 1 of U11
- removed U9: OPA350, symbol JRIX Op Amp:OPA350
- added U6: LT1819, symbol JRIX Op Amp:LT1819
Connections:
- net +5V: now also U6.8 (V-)
- net GNDA: now also U6.8 (V-)
- net at R5.1, R6.2: now also U6.6 (-)
- net at R5.2, U7.5 (+): now also U6.7
- net at R11.2, R9.2: now also U6.5 (+)
- net at R10.2, R12.2: now also U6.3 (+)
- net at R14.2, U7.3 (+): now also U6.1
- net at R13.2, R14.1: now also U6.2 (-)
Other:
- moved on the sheet: C30, C31

Commit message: almost there
Parts:
- removed L2, L4: L_Small, symbol Device:L_Small
- added C1, C2, C34: 1uF, symbol Device:C_Small
- added C28: 100nF, symbol Device:C_Small
- added C29: 220uF, symbol Device:C_Polarized_Small
- added C32: C_Small, symbol Device:C_Small
- added C33: 100n, symbol Device:C_Small
- added C35, C39: 208p, Capacitor_SMD:C_0805_2012Metric_Pad1.18x1.45mm_HandSolder, symbol Device:C_Small
- added C36, C40: 73p6, Capacitor_SMD:C_0805_2012Metric_Pad1.18x1.45mm_HandSolder, symbol Device:C_Small
- added C37, C41: 86p1, Capacitor_SMD:C_0805_2012Metric_Pad1.18x1.45mm_HandSolder, symbol Device:C_Small
- added C38: 30p6, Capacitor_SMD:C_0805_2012Metric_Pad1.18x1.45mm_HandSolder, symbol Device:C_Small
- added R1, R19, R2: 50R, symbol Device:R_Small
- added R15, R16, R17, R23: 10k, symbol Device:R_Small
- added R18, R20, R21, R22, R24, R25, R26, R27, R28, R29, R30, R31: 1k, symbol Device:R_Small
- added U12: REF02Z, Package_DIP:DIP-8_W7.62mm, symbol Reference_Voltage:REF02Z
- added U13, U14: OPA2277-EP, symbol JRIX Op Amp:OPA2277
- added U15, U16, U8: OPA4830, symbol JRIX Op Amp:LT1819
- added U9: OPA350, symbol JRIX Op Amp:OPA350
- C19: value C_Small -> 30p6; footprint (none) -> Capacitor_SMD:C_0805_2012Metric_Pad1.18x1.45mm_HandSolder
- U6: value LT1819 -> OPA4830
Connections:
- net +12V: now also L1.2
- net +5V: now also C33.1, U13.8 (V+)
- net 5VREF: now also U13.6 (-), U13.7
- net DAC1DO: no longer U2.14 (SDO+)
- net DAC1SCK: no longer U2.16 (SCK+)
- net GNDA: now also C19.2, C2.1, C28.2, C29.2, C32.2, C33.2, C34.2, C36.2, C38.2, C40.2, R18.1, R21.1, U12.4 (GND), U13.4 (V-)
- net GNDD: no longer C19.2
- net at C19.1: now also R25.2, U15.3 (+); no longer L1.2
- net at C14.1, C18.1, C21.1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: now also C17.1, C20.1, L3.1, U4.3 (VIN)
- net at C26.1, C27.1, R7.1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: now also U9.3 (+)
- net AAFiltPos: now reaches R10.1
- net AAFiltPos: now also R15.1
- net at R3.1: now also R20.2, U8.1
- net at R4.1: now also R22.2, U8.7
- net AAFiltNeg: now reaches R9.1
- net AAFiltNeg: now also R16.1
- new net: R18.2, R20.1, U8.2 (-)
- new net: C40.1, R31.2, U16.5 (+)
- new net: R21.2, R22.1, U8.6 (-)
- new net: C1.1, R1.1, R2.2
- new net: R19.1, U13.1, U13.2 (-)
- new net: U12.6 (VOUT), U13.3 (+)
- new net: C35.1, R24.2, R25.1
- new net: C35.2, R26.1, U15.1, U15.2 (-)
- new net: R16.2, R23.1, U8.5 (+)
- new net: C34.1, R19.2, U13.5 (+)
- new net: C38.1, R29.2, U16.3 (+)
- new net: C36.1, R27.2, U15.5 (+)
- new net: C39.2, R30.1, U16.1, U16.2 (-)
- new net: R15.2, R17.1, U8.3 (+)
- new net: R17.2, R23.2, U9.2 (-), U9.6
- new net: C41.1, R30.2, R31.1
- new net: C37.1, R26.2, R27.1
- new net: C39.1, R28.2, R29.1
- new net: C2.2, R2.1, U14.5 (+)
- new net: C32.1, L1.1
- new net +12V_FILTERED: C28.1, C29.1, U12.2 (VIN)
- new net DAC2DO: U2.14 (SDO+)
- new net DAC2SCK: U2.16 (SCK+)
- new net VIN: R1.2
- new net VO: C1.2, U14.6 (-), U14.7
- new net V_DUT_NEG: R28.1
- new net V_DUT_NEG_F: C41.2, U16.6 (-), U16.7
- new net V_DUT_POS: R24.1
- new net V_DUT_POS_F: C37.2, U15.6 (-), U15.7
Other:
- note added: "KEEP GNDA, GNDD SEPARATED!"
- moved on the sheet: C22, C23, C24, C25, C30, C31, U10A, U11B, U6C, U7C

Commit message: schematic v1
Parts:
- removed C1, C2: 1uF, symbol Device:C_Small
- removed C15, C16: 100nF, symbol Device:C_Small
- removed C17, C21: 10uF, symbol Device:C_Small
- removed C20, C32: C_Small, symbol Device:C_Small
- removed L3: L_Small, symbol Device:L_Small
- removed R1, R2: 50R, symbol Device:R_Small
- removed U14: OPA2277-EP, symbol JRIX Op Amp:OPA2277
- removed U4: LD1117S25-TR, symbol JRIX Linear Regulator:LD1117S25
- removed U5: LD1117S50-TR, symbol JRIX Linear Regulator:LD1117S50
- added C15, C16, C17, C20, C21, C43, C44, C45, C46, C47: 510uF, symbol Device:C_Polarized_Small
- added C32, C42: 22uF, symbol Device:C_Polarized_Small
- added L2: 1mH, symbol Device:L_Small
- added R32, R33: 1R1, symbol Device:R_Small
- L1: value L_Small -> 1mH
Connections:
- net VDD is gone; now on net +5V: C10.2, C12.2, C3.1, C4.1, C5.1, C6.1, U1.4 (VDD), U2.4 (VDD)
- net +12V_FILTERED: now also C14.1, C18.1, U3.2 (VIN), C15.1, C16.1, C17.1, C20.1, C21.1, C42.1, L2.1
- net GNDA: now also C32.2, C42.2, R32.1, R33.1
- net -12V_FILTERED: now reaches L1.1
- net -12V_FILTERED: now also C32.1, C43.1, C44.1, C45.1, C46.1, C47.1
- net +12V renamed -12V_REG
- net 2V5 renamed +2V5
- net DAC1DO renamed ADC1DO
- net DAC1SCK renamed ADC1SCK
- net DAC2DO renamed ADC2DO
- net DAC2SCK renamed ADC2SCK
- net ~{CNV} renamed ADCCNV
- new net: C15.2, C16.2, C17.2, C20.2, C21.2, R32.2
- new net: C43.2, C44.2, C45.2, C46.2, C47.2, R33.2
- new net +12V_REG: L2.2
Other:
- note removed: "Keep GNDD separated from GNDA Join GNDD and GNDA in star connection away from ADCs"
- moved on the sheet: C13, C14, C18, C19, C28, C29, C34, C35, C36, C37, C38, C39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
