File: PCB/ImpedanceAnalyzer/ImpedanceAnalyzer.kicad_sch (KiCad schematic)
At the start: 0 parts

Commit message: WIP
Other:
- added sheet Supply (Supply.kicad_sch)
Changed lines of the file:
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@@
+		)
+	)
+	(sheet
+		(at 120.015 44.45)
+		(size 20.32 17.78)
+		(fields_autoplaced yes)
+		(stroke
+			(width 0.1524)
+			(type solid)
+		)
+		(fill
+			(color 0 0 0 0.0000)
+		)
+		(property "Sheetname" "Supply"
+			(at 120.015 43.7384 0)
+			(effects
+				(font
+					(size 1.27 1.27)
+				)
+				(justify left bottom)
+			)
+		)
+		(property "Sheetfile" "Supply.kicad_sch"
+			(at 120.015 62.8146 0)
+			(effects
+				(font
+					(size 1.27 1.27)
+				)
+				(justify left top)
+			)
+		)
+		(instances
+			(project "ImpedanceAnalyzer"
+				(path "/08568624-f051-402a-adf3-1b03c2a769ee"
+					(page "3")
+				)
+			)
 		)
 	)
