File: PCB/ImpedanceAnalyzer/ImpedanceAnalyzer.kicad_sch (KiCad schematic)
At the start: 0 parts

Commit message: schematic v1
Parts:
- added GND_LINK2: 0R, symbol Device:R_US
- added J1: CON_+15V, symbol JRIX Connector:6.3-Spade-Con
- added J2: CON_GND, symbol JRIX Connector:6.3-Spade-Con
- added J3: CON_-15V, symbol JRIX Connector:6.3-Spade-Con
- added J4: CON_+5V, symbol JRIX Connector:6.3-Spade-Con
- added J5: Conn_01x04, symbol Connector_Generic:Conn_01x04
- added J6: DUT_H_POT, symbol Connector:Conn_Coaxial_Small
- added J7: DUT_L_POT, symbol Connector:Conn_Coaxial_Small
- added J8: DUT_H_CUR, symbol Connector:Conn_Coaxial_Small
- added J9: DUT_L_CUR, symbol Connector:Conn_Coaxial_Small
Connections:
- new net ADC Range/DUT_H_POT: J6.1 (In)
- new net ADC Range/DUT_L_POT: J7.1 (In)
- new net ADC Range/GNDA: GND_LINK2.1, J6.2 (Ext), J7.2 (Ext), J8.2 (Ext), J9.2 (Ext)
- new net ADC Range/GNDD: GND_LINK2.2
- new net DAC Power Amp/DUT_L_CUR: J9.1 (In)
- new net Digital/+5V_MW_REG: J4.1, J4.2, J5.1 (Pin_1)
- new net RX: J5.3 (Pin_3)
- new net Range Select/DUT_H_CUR: J8.1 (In)
- new net Supply/+15V_MW: J1.1, J1.2
- new net Supply/-15V_MW: J3.1, J3.2
- new net Supply/GND_MW: J2.1, J2.2, J5.2 (Pin_2)
- new net TX: J5.4 (Pin_4)
Other:
- sheet Analog Front End renamed ADC
- added sheet ADC Range (ADC_RANGE.kicad_sch)
- added sheet DAC (DAC.kicad_sch)
- added sheet DAC Power Amp (DAC_POWER_AMP.kicad_sch)
- added sheet Digital (digital.kicad_sch)
- added sheet Range Select (RANGE_SELECT.kicad_sch)
- sheet ADC: file ANFE.kicad_sch -> ADC.kicad_sch
- sheet ADC ports: added +12V_FILTERED, +2V5_REG, +5V_REG, +6V_REG, -1V_REG, -5V_REG, ADC1MISO, ADC1SCK, ADC2MISO, ADC2SCK, ADCCNV, GNDA, GNDD, I_DUT_NEG, I_DUT_POS, V_DUT_NEG, V_DUT_POS; removed none
- sheet Supply ports: added +12V_FILTERED, +15V_MW, +3V3_REG, +5V_REG, +6V_REG, -12V_FILTERED, -15V_MW, -1V_REG, -5V_REG, GNDA, GNDD, GND_MW; removed none
- note added: "4x 6.3-Spade-Con"
- note added: "ANALOG/DIGITAL GROUND LINK"
- note added: "KELVIN BRIDGE"
- note added: "MEAN WELL RT65C"
- note added: "Nextion Display"

Commit message: ready for pcb
Parts:
- removed J1: CON_+15V, symbol JRIX Connector:6.3-Spade-Con
- removed J2: CON_GND, symbol JRIX Connector:6.3-Spade-Con
- removed J3: CON_-15V, symbol JRIX Connector:6.3-Spade-Con
- removed J4: CON_+5V, symbol JRIX Connector:6.3-Spade-Con
- added J1, J10, J2, J3: 63849-1, JRIX FASTON Connectors Footprints:TE_63849-1, symbol JRIX FASTON Connector:63849-1
- GND_LINK2: footprint (none) -> JRIX Resistor SMD:Resistor SMD - 2818
- J5: footprint (none) -> Connector_JST:JST_XH_B4B-XH-A_1x04_P2.50mm_Vertical
- J6, J7, J8, J9: footprint (none) -> Connector_Coaxial:BNC_TEConnectivity_1478204_Vertical
Connections:
- net Digital/+5V_MW_REG renamed +5V_MW
- net +5V_MW: now also J3.1_1, J3.1_2
- net Supply/GND_MW renamed GND_MW
- net GND_MW: now also J1.1_1, J1.1_2
- new net +15V_MW: J10.1_1, J10.1_2
- new net -15V_MW: J2.1_1, J2.1_2
Other:
- note added: "CON_+15V"
- note added: "CON_+5V"
- note added: "CON_-15V"
- note added: "CON_GND"
- note removed: "4x 6.3-Spade-Con"

Commit message: corrected kicad
Connections:
- net ADC Range/GNDD is gone; now on net ADC Range/GNDA: GND_LINK2.2
Other:
- sheet DAC ports: added +5V_REG, -5V_REG; removed none
- sheet DAC Power Amp ports: added +5V_REG, -5V_REG, GNDA; removed none
- sheet Supply ports: added +2V5_REG, +5V_MW; removed none
- moved on the sheet: GND_LINK2

Commit message: pcb 90%
Other:
- moved on the sheet: GND_LINK2
Changed lines of the file:
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@@
 	)
 	(junction
-		(at 120.65 130.81)
+		(at 123.19 130.81)
 		(diameter 0)
 		(color 0 0 0 0)
@@
 	)
 	(junction
+		(at 123.19 81.28)
+		(diameter 0)
+		(color 0 0 0 0)
+	)
+	(junction
 		(at 17.78 48.26)
 		(diameter 0)
@@
 	)
 	(junction
-		(at 120.65 82.55)
-		(diameter 0)
-		(color 0 0 0 0)
-	)
-	(junction
 		(at 127 64.77)
 		(diameter 0)
@@
 	)
 	(junction
-		(at 120.65 154.94)
+		(at 124.46 153.67)
 		(diameter 0)
 		(color 0 0 0 0)
@@
 	)
 	(junction
-		(at 123.19 81.28)
+		(at 66.04 82.55)
 		(diameter 0)
 		(color 0 0 0 0)
 	)
 	(junction
-		(at 66.04 82.55)
+		(at 176.53 132.08)
 		(diameter 0)
 		(color 0 0 0 0)
 	)
 	(junction
-		(at 123.19 130.81)
+		(at 107.95 138.43)
 		(diameter 0)
 		(color 0 0 0 0)
 	)
 	(junction
-		(at 176.53 132.08)
+		(at 134.62 148.59)
 		(diameter 0)
 		(color 0 0 0 0)
 	)
 	(junction
-		(at 107.95 138.43)
+		(at 120.65 82.55)
 		(diameter 0)
 		(color 0 0 0 0)
 	)
 	(junction
-		(at 134.62 148.59)
+		(at 134.62 153.67)
 		(diameter 0)
 		(color 0 0 0 0)
 	)
 	(junction
-		(at 104.14 139.7)
+		(at 120.65 153.67)
 		(diameter 0)
 		(color 0 0 0 0)
 	)
 	(junction
-		(at 265.43 83.82)
+		(at 104.14 139.7)
 		(diameter 0)
 		(color 0 0 0 0)
 	)
 	(junction
-		(at 123.19 128.27)
+		(at 265.43 83.82)
 		(diameter 0)
 		(color 0 0 0 0)
@@
 	(wire
 		(pts
-			(xy 120.65 130.81) (xy 123.19 130.81)
+			(xy 265.43 50.8) (xy 264.16 50.8)
 		)
 		(stroke
@@
 	(wire
 		(pts
-			(xy 265.43 50.8) (xy 264.16 50.8)
+			(xy 118.11 41.91) (xy 142.24 41.91)
 		)
 		(stroke
@@
 	(wire
 		(pts
-			(xy 118.11 41.91) (xy 142.24 41.91)
+			(xy 220.98 55.88) (xy 246.38 55.88)
 		)
 		(stroke
@@
 	(wire
 		(pts
-			(xy 220.98 55.88) (xy 246.38 55.88)
+			(xy 185.42 53.34) (xy 199.39 53.34)
 		)
 		(stroke
@@
 	(wire
 		(pts
-			(xy 185.42 53.34) (xy 199.39 53.34)
+			(xy 25.4 119.38) (xy 27.94 119.38)
 		)
 		(stroke
@@
 	(wire
 		(pts
-			(xy 25.4 119.38) (xy 27.94 119.38)
+			(xy 86.36 83.82) (xy 86.36 27.94)
 		)
 		(stroke
@@
 	(wire
 		(pts
-			(xy 86.36 83.82) (xy 86.36 27.94)
+			(xy 134.62 153.67) (xy 134.62 156.21)
 		)
 		(stroke
@@
 	(wire
 		(pts
+			(xy 120.65 153.67) (xy 120.65 158.75)
+		)
+		(stroke
+			(width 0)
+			(type default)
+		)
+	)
+	(wire
+		(pts
 			(xy 53.34 92.71) (xy 57.15 92.71)
 		)
@@
 	(wire
 		(pts
-			(xy 134.62 148.59) (xy 134.62 154.94)
+			(xy 134.62 148.59) (xy 134.62 153.67)
 		)
 		(stroke
@@
 	(wire
 		(pts
-			(xy 133.35 154.94) (xy 134.62 154.94)
+			(xy 133.35 153.67) (xy 134.62 153.67)
 		)
 		(stroke
@@
 	(wire
 		(pts
-			(xy 123.19 81.28) (xy 123.19 128.27)
+			(xy 120.65 82.55) (xy 120.65 133.35)
 		)
 		(stroke
@@
 	(wire
 		(pts
-			(xy 120.65 154.94) (xy 125.73 154.94)
+			(xy 120.65 153.67) (xy 124.46 153.67)
 		)
 		(stroke
@@
 	(wire
 		(pts
-			(xy 120.65 133.35) (xy 120.65 154.94)
+			(xy 120.65 133.35) (xy 120.65 153.67)
 		)
 		(stroke
@@
 	(wire
 		(pts
-			(xy 120.65 158.75) (xy 120.65 154.94)
-		)
-		(stroke
-			(width 0)
-			(type default)
-		)
-	)
-	(wire
-		(pts
 			(xy 124.46 62.23) (xy 124.46 30.48)
 		)
@@
 	(wire
 		(pts
+			(xy 134.62 156.21) (xy 124.46 156.21)
+		)
+		(stroke
+			(width 0)
+			(type default)
+		)
+	)
+	(wire
+		(pts
 			(xy 186.69 67.31) (xy 186.69 33.02)
 		)
@@
 	(wire
 		(pts
+			(xy 124.46 153.67) (xy 124.46 156.21)
+		)
+		(stroke
+			(width 0)
+			(type default)
+		)
+	)
+	(wire
+		(pts
 			(xy 179.07 120.65) (xy 175.26 120.65)
 		)
@@
 	(wire
 		(pts
-			(xy 120.65 82.55) (xy 120.65 130.81)
-		)
-		(stroke
-			(width 0)
-			(type default)
-		)
-	)
-	(wire
-		(pts
 			(xy 142.24 54.61) (xy 139.7 54.61)
 		)
@@
 	(wire
 		(pts
-			(xy 116.84 130.81) (xy 120.65 130.81)
+			(xy 116.84 130.81) (xy 123.19 130.81)
 		)
 		(stroke
@@
 	(wire
 		(pts
-			(xy 123.19 128.27) (xy 123.19 130.81)
-		)
-		(stroke
-			(width 0)
-			(type default)
-		)
-	)
-	(wire
-		(pts
 			(xy 121.92 25.4) (xy 121.92 57.15)
 		)
@@
 	(wire
 		(pts
+			(xy 123.19 81.28) (xy 123.19 130.81)
+		)
+		(stroke
+			(width 0)
+			(type default)
+		)
+	)
+	(wire
+		(pts
 			(xy 133.35 67.31) (xy 133.35 24.13)
 		)
@@
 	(wire
 		(pts
-			(xy 120.65 130.81) (xy 120.65 133.35)
-		)
-		(stroke
-			(width 0)
-			(type default)
-		)
-	)
-	(wire
-		(pts
 			(xy 85.09 163.83) (xy 104.14 163.83)
 		)
@@
 	(wire
 		(pts
-			(xy 116.84 128.27) (xy 123.19 128.27)
-		)
-		(stroke
-			(width 0)
-			(type default)
-		)
-	)
-	(wire
-		(pts
 			(xy 93.98 148.59) (xy 123.19 148.59)
 		)
@@
 	(wire
 		(pts
+			(xy 124.46 153.67) (xy 125.73 153.67)
+		)
+		(stroke
+			(width 0)
+			(type default)
+		)
+	)
+	(wire
+		(pts
 			(xy 127 33.02) (xy 127 64.77)
 		)
@@
 	(wire
 		(pts
-			(xy 123.19 128.27) (xy 142.24 128.27)
+			(xy 116.84 128.27) (xy 142.24 128.27)
 		)
 		(stroke
@@
 	(symbol
 		(lib_id "Device:R_US")
-		(at 129.54 154.94 90)
+		(at 129.54 153.67 90)
 		(unit 1)
 		(exclude_from_sim no)
@@
 		(dnp no)
 		(property "Reference" "GND_LINK2"
-			(at 129.54 150.876 90)
+			(at 129.54 149.606 90)
 			(effects
 				(font
@@
 		)
 		(property "Value" "0R"
-			(at 129.54 152.654 90)
+			(at 129.54 151.384 90)
 			(effects
 				(font
@@
 		)
 		(property "Footprint" "JRIX Resistor SMD:Resistor SMD - 2818"
-			(at 129.794 153.924 90)
+			(at 129.794 152.654 90)
 			(effects
 				(font
@@
 		)
 		(property "Datasheet" "~"
-			(at 129.54 154.94 0)
+			(at 129.54 153.67 0)
 			(effects
 				(font
@@
 		)
 		(property "Description" "Resistor, US symbol"
-			(at 129.54 154.94 0)
+			(at 129.54 153.67 0)
 			(effects
 				(font

Commit message: PCB done
Connections:
- net ADC Range/GNDA: now also J5.2 (Pin_2)
- net GND_MW: no longer J5.2 (Pin_2)
Changed lines of the file:
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@@
+	)
+	(junction
+		(at 187.96 99.06)
+		(diameter 0)
+		(color 0 0 0 0)
 	)
 	(junction
@@
 		(color 0 0 0 0)
 	)
-	(junction
-		(at 251.46 78.74)
-		(diameter 0)
-		(color 0 0 0 0)
-	)
 	(bus_entry
 		(at 179.07 118.11)
@@
 	(wire
 		(pts
+			(xy 187.96 99.06) (xy 266.7 99.06)
+		)
+		(stroke
+			(width 0)
+			(type default)
+		)
+	)
+	(wire
+		(pts
 			(xy 134.62 64.77) (xy 134.62 22.86)
 		)
@@
 	(wire
 		(pts
-			(xy 251.46 78.74) (xy 251.46 99.06)
-		)
-		(stroke
-			(width 0)
-			(type default)
-		)
-	)
-	(wire
-		(pts
 			(xy 85.09 25.4) (xy 85.09 85.09)
 		)
@@
 	(wire
 		(pts
-			(xy 266.7 99.06) (xy 251.46 99.06)
-		)
-		(stroke
-			(width 0)
-			(type default)
-		)
-	)
-	(wire
-		(pts
 			(xy 120.65 133.35) (xy 120.65 153.67)
 		)
@@
 	(wire
 		(pts
+			(xy 187.96 99.06) (xy 187.96 74.93)
+		)
+		(stroke
+			(width 0)
+			(type default)
+		)
+	)
+	(wire
+		(pts
 			(xy 90.17 101.6) (xy 96.52 101.6)
 		)
@@
 	(wire
 		(pts
-			(xy 187.96 132.08) (xy 187.96 74.93)
+			(xy 187.96 132.08) (xy 187.96 99.06)
 		)
 		(stroke
@@
 	)
 	(label "RX"
-		(at 262.8907 101.6 0)
+		(at 262.8907 101.6 180)
 		(fields_autoplaced yes)
 		(effects
@@
 				(size 1.27 1.27)
 			)
-			(justify left bottom)
-		)
-	)
+			(justify right bottom)
+		)
+	)
