File: PCB/ImpedanceAnalyzer/ADC_RANGE.kicad_sch (KiCad schematic)
At the start: 32 parts, among them U25 PGA855, U26 PGA855, U28 ILQ1, U29 ILQ1

Commit message: ready for pcb
Parts:
- removed C161, C164, C167, C170, C176, C177: 220uF, symbol Device:C_Polarized_Small
- removed U25, U26: PGA855, symbol JRIX Programmable Amplifiers:PGA855
- removed U28, U29: ILQ1, symbol JRIX Optocouplers:ILQ1
- added C161, C164, C167, C170, C176, C177: 1uF, Capacitor_SMD:C_0805_2012Metric_Pad1.18x1.45mm_HandSolder, symbol Device:C_Small
- added U25, U35: PGA855, Package_DFN_QFN:VQFN-16-1EP_3x3mm_P0.5mm_EP1.45x1.45mm, symbol JRIX PGA:PGA855RGTR
- added U31, U33: ILQ1, Package_DIP:DIP-16_W7.62mm, symbol JRIX Optocouplers:ILQ1
- C162, C165, C168, C171, C174, C175: footprint (none) -> Capacitor_SMD:C_0805_2012Metric_Pad1.18x1.45mm_HandSolder
- C163, C166, C169, C172: footprint (none) -> Capacitor_THT:C_Disc_D3.4mm_W2.1mm_P2.50mm
- R86, R87, R88, R89, R90, R91, R92, R93, R94, R95, R96, R97: footprint (none) -> Resistor_SMD:R_0805_2012Metric_Pad1.20x1.40mm_HandSolder
Connections:
- net +12V_FILTERED: now also C164.1, C170.1, C176.1, C177.1, U25.6 (VS+), U25.7 (LVDD), U35.6 (VS+), U35.7 (LVDD)
- net -12V_FILTERED: now also C161.1, C167.1, U25.14 (LVSS), U25.15 (VS-), U35.14 (LVSS), U35.15 (VS-)
- net DUT_H_POT: now also U35.3 (IN-)
- net DUT_I_SENSE_+: now also U25.3 (IN-)
- net DUT_I_SENSE_-: now also U25.2 (IN+)
- net DUT_L_POT: now also U35.2 (IN+)
- net GNDA: now also C161.2, C164.2, C167.2, C170.2, C176.2, C177.2, U25.13 (VOCM), U25.16 (DGND), U31.10, U31.12, U31.13, U31.16, U31.9, U33.10, U33.12, U33.13, U33.16, U33.9, U35.13 (VOCM), U35.16 (DGND)
- net GNDD: now also U31.2, U31.3, U31.6, U31.7, U31.8, U33.2, U33.3, U33.6, U33.7, U33.8
- net I_DUT_NEG: now also U25.11 (OUT-)
- net I_DUT_POS: now also U25.10 (OUT+)
- net V_DUT_NEG: now also U35.11 (OUT-)
- net V_DUT_POS: now also U35.10 (OUT+)
- net at R88.1: now also U31.5
- net at R92.1: now also U25.4 (A0), U33.11
- net at R86.1: now also U31.1
- net at R89.1: now also U31.15, U35.1 (A2)
- net at R87.1: now also U31.4
- net at R90.1: now also U31.14, U35.5 (A1)
- net at R93.1: now also U25.5 (A1), U33.14
- net at R97.1: now also U33.5
- net at R91.1: now also U31.11, U35.4 (A0)
- net at R96.1: now also U33.4
- net at R95.1: now also U33.1
- net at R94.1: now also U25.1 (A2), U33.15
Other:
- moved on the sheet: C165, C166

Commit message: corrected kicad
Changed lines of the file:
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@@
 		(on_board yes)
 		(dnp no)
-		(fields_autoplaced yes)
 		(property "Reference" "#PWR087"
 			(at 167.64 91.44 0)
@@
 		)
 		(property "Value" "GNDA"
-			(at 167.64 90.17 0)
+			(at 170.434 88.9 0)
 			(effects
 				(font
