File: PCB/ImpedanceAnalyzer/DAC.kicad_sch (KiCad schematic)
At the start: 89 parts, among them U14 OPA4830, U16 OPA4830, U17 OPA4830, U6 LTC1668CG

Commit message: ready for pcb
Parts:
- removed U16: OPA4830, symbol JRIX Op Amp:OPA4830
- added unit 5 of U17
- C100, C101: value 10p5 -> 10p; footprint (none) -> Capacitor_THT:C_Disc_D3.0mm_W2.0mm_P2.50mm
- C102, C103, C104, C105: footprint (none) -> Capacitor_THT:C_Disc_D4.7mm_W2.5mm_P5.00mm
- C106, C107, C110, C111, C114, C115, C98, C99: value 10p -> 8p2; footprint (none) -> Capacitor_THT:C_Disc_D3.4mm_W2.1mm_P2.50mm
- C108, C109: value 16p2 -> 15p; footprint (none) -> Capacitor_THT:C_Disc_D3.4mm_W2.1mm_P2.50mm
- C112, C113: value 19p6 -> 18p; footprint (none) -> Capacitor_THT:C_Disc_D3.4mm_W2.1mm_P2.50mm
- C116, C117: value 20p5 -> 22p; footprint (none) -> Capacitor_THT:C_Disc_D3.4mm_W2.1mm_P2.50mm
- C118, C119, C124, C125: footprint (none) -> Capacitor_THT:CP_Radial_D6.3mm_P2.50mm
- C120, C121, C126, C127, C96, C97: footprint (none) -> Capacitor_SMD:C_0805_2012Metric_Pad1.18x1.45mm_HandSolder
- C122, C123, C128, C129: footprint (none) -> Capacitor_THT:C_Disc_D3.4mm_W2.1mm_P2.50mm
- L3: footprint (none) -> Inductor_THT:L_CommonMode_Wuerth_WE-CMB-L
- L4, L5: footprint (none) -> Inductor_THT:L_Axial_L14.5mm_D5.8mm_P20.32mm_Horizontal_Fastron_HBCC
- L6, L7: footprint (none) -> Inductor_THT:L_Axial_L9.5mm_D4.0mm_P12.70mm_Horizontal_Fastron_SMCC
- R43, R44, R45, R46, R47, R48, R49, R50, R51, R52, R53, R54, R55, R56, R57, R58, R59, R60, R61, R62, R63, R64, R65, R66, R67, R68, R69, R70, R71, R72, R73, R74, R75, R76, R77, R78: footprint (none) -> Resistor_THT:R_Axial_DIN0207_L6.3mm_D2.5mm_P10.16mm_Horizontal
- U14, U17: footprint (none) -> Package_SO:TSSOP-14_4.4x5mm_P0.65mm
Connections:
- net +5V: now also U17.4 (V+)
- net -5V: now also U17.11 (V-)
- net VOUT+: now also L3.2 (1); no longer L3.1
- net VOUT-: now also L3.4 (2); no longer L3.2
- net at L4.1: now also L3.9 (3); no longer L3.3
- net at R54.1: now also C101.2, R52.1, U17.7
- net at L5.1: now also L3.7 (4); no longer L3.4

Commit message: corrected kicad
Connections:
- net +5V renamed +5V_REG
- net -5V renamed -5V_REG
Changed lines of the file:
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@@
+	(wire
+		(pts
+			(xy 359.41 139.7) (xy 367.03 139.7)
+		)
+		(stroke
+			(width 0)
+			(type default)
+		)
+	)
 	(wire
 		(pts
@@
 		(pts
 			(xy 289.56 27.94) (xy 289.56 40.64)
+		)
+		(stroke
+			(width 0)
+			(type default)
+		)
+	)
+	(wire
+		(pts
+			(xy 359.41 142.24) (xy 367.03 142.24)
 		)
 		(stroke
@@
 		)
 	)
+	(label "-5V"
+		(at 359.41 142.24 0)
+		(fields_autoplaced yes)
+		(effects
+			(font
+				(size 1.27 1.27)
+			)
+			(justify left bottom)
+		)
+	)
 	(label "VOUT+"
 		(at 143.51 146.05 0)
@@
 	(label "-5V"
 		(at 45.72 173.99 0)
+		(fields_autoplaced yes)
+		(effects
+			(font
+				(size 1.27 1.27)
+			)
+			(justify left bottom)
+		)
+	)
+	(label "+5V"
+		(at 359.41 139.7 0)
 		(fields_autoplaced yes)
 		(effects
@@
 		)
 	)
+	(hierarchical_label "-5V_REG"
+		(shape input)
+		(at 367.03 142.24 0)
+		(fields_autoplaced yes)
+		(effects
+			(font
+				(size 1.27 1.27)
+			)
+			(justify left)
+		)
+	)
+	(hierarchical_label "+5V_REG"
+		(shape input)
+		(at 367.03 139.7 0)
+		(fields_autoplaced yes)
+		(effects
+			(font
+				(size 1.27 1.27)
+			)
+			(justify left)
+		)
+	)
