File: PCB/ImpedanceAnalyzer/ADC.kicad_sch (KiCad schematic)
At the start: 106 parts, among them U1 LTC2311, U11 OPA4830, U12 REF02Z, U13 OPA2277-EP, U2 LTC2311, U3 LT1819, U4 LT1819, U5 OPA350, U7 OPA350, U8 OPA4830, U9 OPA4830

Commit message: ready for pcb
Parts:
- removed C14, C23, C25, C30, C31, C48, C50, C61, C64, C66, C71, C79, C80: 100u, symbol Device:C_Polarized_Small
- added C14, C23, C25, C30, C31, C48, C50, C61, C64, C66, C71, C79, C80: 1uF, Capacitor_SMD:C_0805_2012Metric_Pad1.18x1.45mm_HandSolder, symbol Device:C_Small
- added C199, C200, C201, C202: 8p, Capacitor_SMD:C_0603_1608Metric_Pad1.08x0.95mm_HandSolder, symbol Device:C_Small
- added C203, C204, C205, C206: 5p6, Capacitor_SMD:C_0603_1608Metric_Pad1.08x0.95mm_HandSolder, symbol Device:C_Small
- added C207, C208, C209, C210: 30p, Capacitor_SMD:C_0603_1608Metric_Pad1.08x0.95mm_HandSolder, symbol Device:C_Small
- C13, C18, C22, C24, C33, C63, C65: value 100n -> 100nF; footprint (none) -> Capacitor_SMD:C_0805_2012Metric_Pad1.18x1.45mm_HandSolder
- C19, C38, C51, C52: value 30p6 -> 30p; footprint Capacitor_SMD:C_0805_2012Metric_Pad1.18x1.45mm_HandSolder -> Capacitor_SMD:C_0603_1608Metric_Pad1.08x0.95mm_HandSolder
- C26, C28, C34, C49, C62, C75, C76, C81, C82, C85, C87: footprint (none) -> Capacitor_SMD:C_0805_2012Metric_Pad1.18x1.45mm_HandSolder
- C27: footprint (none) -> Capacitor_SMD:C_1206_3216Metric_Pad1.33x1.80mm_HandSolder
- C29: value 220uF -> 470uF; footprint (none) -> Capacitor_THT:CP_Radial_D10.0mm_P5.00mm
- C35, C39, C53, C54: value 208p -> 200p; footprint Capacitor_SMD:C_0805_2012Metric_Pad1.18x1.45mm_HandSolder -> Capacitor_SMD:C_0603_1608Metric_Pad1.08x0.95mm_HandSolder
- C36, C40, C55, C56: value 73p6 -> 68p; footprint Capacitor_SMD:C_0805_2012Metric_Pad1.18x1.45mm_HandSolder -> Capacitor_SMD:C_0603_1608Metric_Pad1.08x0.95mm_HandSolder
- C37, C41, C57, C58: value 86p1 -> 56p; footprint Capacitor_SMD:C_0805_2012Metric_Pad1.18x1.45mm_HandSolder -> Capacitor_SMD:C_0603_1608Metric_Pad1.08x0.95mm_HandSolder
- C59, C60, C67, C68, C69, C70, C72, C73, C74, C77, C78, C83, C84: footprint (none) -> Capacitor_THT:C_Disc_D3.4mm_W2.1mm_P2.50mm
- C7: value 100u -> 100uF; footprint (none) -> Capacitor_THT:CP_Radial_D6.3mm_P2.50mm
- C86: footprint (none) -> Capacitor_THT:CP_Radial_D6.3mm_P2.50mm
- R10, R11, R12, R15, R16, R17, R19, R23, R7, R8, R9: footprint (none) -> Resistor_SMD:R_0805_2012Metric_Pad1.20x1.40mm_HandSolder
- R114, R24, R25, R26, R27, R5: footprint (none) -> Resistor_THT:R_Array_SIP8
- U11, U8, U9: footprint (none) -> Package_SO:TSSOP-14_4.4x5mm_P0.65mm
- U13, U5, U7: footprint (none) -> Package_DIP:DIP-8_W7.62mm
- U3, U4: footprint (none) -> Package_SO:SOIC-8_3.9x4.9mm_P1.27mm
Connections:
- net +5V_REG: now also C25.1, C30.1, C48.2, C50.1, C71.1, C79.1
- net +6V_REG: now also C14.1, C23.1
- net -1V_REG: now also U3.4 (V-), U4.4 (V-), C64.2, C66.2; no longer U3.8 (V-), U4.8 (V-)
- net -5V_REG: now also C31.2, C61.2, C80.2
- net GNDA: now also C38.1, C40.1, C52.1, C56.1, C14.2, C203.2, C204.1, C205.2, C206.1, C23.2, C25.2, C30.2, C31.1, C48.1, C50.2, C61.1, C64.1, C66.1, C71.2, C79.2, C80.1; no longer C38.2, C40.2, C52.2, C56.2
- net at C55.1, R26.6, U8.10 (+): now also C203.1
- net at C57.2, R15.1, U8.8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: now also C209.2
- net at R24.8, U8.5 (+): now also C40.2, C206.2; no longer C40.1
- net at C41.2, R9.1, U8.6 (-)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: now also C208.2
- net at C35.2, R24.1, U11.1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: now also C200.2
- net at C41.1, R24.4, R24.7: now also C208.1
- net at C37.2, R10.1, U8.1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: now also C207.2
- net at C36.1, R24.6, U8.3 (+): now also C205.1
- net at C57.1, R26.2, R26.5: now also C209.1
- net at C53.2, R26.1, U11.8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: now also C201.2
- net at R25.8, U11.12 (+): now also C52.2; no longer C52.1
- net at C54.2, R26.3, U11.13 (-)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: now also C202.2
- net at C35.1, R114.2, R114.5: now also C200.1
- net at C53.1, R25.2, R25.5: now also C201.1
- net at C58.2, R16.1, U8.13 (-)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: now also C210.2
- net at C37.1, R24.2, R24.5: now also C207.1
- net at C39.1, R114.4, R114.7: now also C199.1
- net at R114.8, U11.5 (+): now also C38.2; no longer C38.1
- net at C39.2, R24.3, U11.6 (-)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: now also C199.2
- net at C58.1, R26.4, R26.7: now also C210.1
- net at R26.8, U8.12 (+): now also C56.2, C204.2; no longer C56.1
- net at C54.1, R25.4, R25.7: now also C202.1

Commit message: corrected kicad
Parts:
- removed C27: 4u7, Capacitor_SMD:C_1206_3216Metric_Pad1.33x1.80mm_HandSolder, symbol Device:C_Polarized_Small
- added C27: 4u7, Capacitor_SMD:C_1206_3216Metric_Pad1.33x1.80mm_HandSolder, symbol Device:C_Small
Connections:
- net GNDA: now also R27.1, R27.3, C27.1; no longer R5.5, R5.7
- net I_DUT_NEG: now also R114.7; no longer R25.3
- net I_DUT_POS: now also R114.5; no longer R25.1
- net at U4.5 (+), U9.14: now also R5.7; no longer R5.4
- net at C210.1, C58.1, R26.7: now also R24.8; no longer R26.4
- net at C206.2, C40.2, U8.5 (+): now also R26.4; no longer R24.8
- net at C19.1, U11.3 (+): now also R25.2; no longer R114.6
- net at C208.1, C41.1, R24.4: now also R26.3; no longer R24.7
- net at C205.1, C36.1, U8.3 (+): now also R26.2; no longer R24.6
- net at C209.1, C57.1, R26.5: now also R24.6; no longer R26.2
- net at C201.2, C53.2, U11.8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: now also R24.5; no longer R26.1
- net at C202.2, C54.2, U11.13 (-)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: now also R24.7; no longer R26.3
- net at C200.1, C35.1, R114.2: now also R25.1; no longer R114.5
- net at U3.3 (+), U9.1: now also R5.2; no longer R27.2
- net at U4.3 (+), U9.8: now also R5.5; no longer R5.2
- net at C201.1, C53.1, R25.5: now also R114.6; no longer R25.2
- net at C207.1, C37.1, R24.2: now also R26.1; no longer R24.5
- net at C199.1, C39.1, R114.4: now also R25.3; no longer R114.7
- net at C38.2, U11.5 (+): now also R25.4; no longer R114.8
- net at U3.5 (+), U9.7: now also R5.4; no longer R27.4
- net at C26.1, R7.1, R8.2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: now also C27.2
- net at R5.6, U9.9 (-): now also R27.6; no longer R5.1
- net at C202.1, C54.1, R25.7: now also R114.8; no longer R25.4
- net at R5.8, U9.13 (-): now also R27.8; no longer R5.3
- new net: R27.2, R5.1, U9.2 (-)
- new net: R27.4, R5.3, U9.6 (-)
Other:
- moved on the sheet: C11, C9, R114C, R114D, R26A, R26B

Commit message: pcb 90%
Parts:
- removed C29: 470uF, Capacitor_THT:CP_Radial_D10.0mm_P5.00mm, symbol Device:C_Polarized_Small
- removed C3, C4, C7: 100uF, Capacitor_THT:CP_Radial_D6.3mm_P2.50mm, symbol Device:C_Polarized_Small
- removed C59, C60, C67, C68: 100pF, Capacitor_THT:C_Disc_D3.4mm_W2.1mm_P2.50mm, symbol Device:C_Small
- removed C86: 100u, Capacitor_THT:CP_Radial_D6.3mm_P2.50mm, symbol Device:C_Polarized_Small
- added C29, C3, C4, C7, C86: 100uF, Capacitor_SMD:C_1206_3216Metric_Pad1.33x1.80mm_HandSolder, symbol Device:C_Small
Connections:
- net +12V_FILTERED: now also C29.1
- net +2V5_REG: now also C7.1, C86.1
- net +5V_REG: now also C3.1, C4.1
- net GNDA: now also C29.2, C3.2, C4.2
- net GNDD: now also C7.2, C86.2
