File: PCB/ImpedanceAnalyzer/RANGE_SELECT.kicad_sch (KiCad schematic)
At the start: 57 parts, among them K1 RY-12W-K, K2 RY-12W-K, K3 RY-12W-K, K4 RY-12W-K, K5 RY-12W-K, K6 RY-12W-K, K7 RY-12W-K, U28 ILQ1, U29 ILQ1, U30 ILQ1, U31 ILQ1, U32 MUX-24, U33 ILQ1

Commit message: ready for pcb
Parts:
- removed C178, C179, C180, C181, C183, C184, C185: 220uF, symbol Device:C_Polarized_Small
- removed U28, U29, U31, U33: ILQ1, symbol JRIX Optocouplers:ILQ1
- added C178, C179, C180, C181, C183, C184, C185: 1uF, Capacitor_SMD:C_0805_2012Metric_Pad1.18x1.45mm_HandSolder, symbol Device:C_Small
- added U16, U26: ILQ1, Package_DIP:DIP-16_W7.62mm, symbol JRIX Optocouplers:ILQ1
- C182, C186: footprint (none) -> Capacitor_SMD:C_0805_2012Metric_Pad1.18x1.45mm_HandSolder
- K1, K2, K3, K4, K5, K6, K7: value RY-12W-K -> RY-12W-K; footprint (none) -> JRIX Relay Footprints:RELAY_RY-12W-K
- R100, R101, R102, R103, R104, R105, R106, R107, R108, R109, R110, R98, R99: footprint (none) -> Resistor_SMD:R_0805_2012Metric_Pad1.20x1.40mm_HandSolder
- R105_RANGE1: renamed from R105_RANGE; footprint (none) -> Resistor_THT:R_Axial_DIN0516_L15.5mm_D5.0mm_P20.32mm_Horizontal
- R106_RANGE1: renamed from R106_RANGE; footprint (none) -> Resistor_THT:R_Axial_DIN0207_L6.3mm_D2.5mm_P10.16mm_Horizontal
- R107_RANGE1: renamed from R107_RANGE; footprint (none) -> Resistor_THT:R_Axial_DIN0207_L6.3mm_D2.5mm_P10.16mm_Horizontal
- R108_RANGE1: renamed from R108_RANGE; footprint (none) -> Resistor_THT:R_Axial_DIN0207_L6.3mm_D2.5mm_P10.16mm_Horizontal
- R109_RANGE1: renamed from R109_RANGE; footprint (none) -> Resistor_THT:R_Axial_DIN0207_L6.3mm_D2.5mm_P10.16mm_Horizontal
- R110_RANGE1: renamed from R110_RANGE; footprint (none) -> Resistor_THT:R_Axial_DIN0207_L6.3mm_D2.5mm_P10.16mm_Horizontal
- R111, R112, R113, R115, R116, R117, R118, R119: footprint (none) -> Resistor_THT:R_Axial_DIN0207_L6.3mm_D2.5mm_P10.16mm_Horizontal
- R111_RANGE1: renamed from R111_RANGE; footprint (none) -> Resistor_THT:R_Axial_DIN0207_L6.3mm_D2.5mm_P10.16mm_Horizontal
- U30, U32: footprint (none) -> Package_DIP:DIP-16_W7.62mm
Connections:
- net +12V_FILTERED: now also K1.16, K2.16, K3.16, K4.16, K5.16, K6.16, K7.16, C178.1, C179.1, C180.1, C181.1, C183.1, C184.1, C185.1; no longer K1.1, K2.1, K3.1, K4.1, K5.1, K6.1, K7.1
- net GNDA: now also C178.2, C179.2, C180.2, C181.2, C183.2, C184.2, C185.2, U16.10, U16.12, U16.13, U16.16, U16.7, U16.8, U16.9, U26.10, U26.12, U26.13, U26.16, U26.7, U26.8, U26.9; no longer U30.10, U30.7, U30.8
- net GNDD: now also U30.7, U16.2, U16.3, U16.6, U26.2, U26.3, U26.6
- net at R111_RANGE1.2: now also K1.4; no longer K1.7
- net at R103.1: now also U30.8; no longer U30.4
- net at R99.1: now also U26.4
- net at R105_RANGE1.2: now also K2.4; no longer K2.7
- net at K4.4: now also R107_RANGE1.2
- net at D9.2 (A), U30.11: now also K4.1; no longer K4.8
- net at R106_RANGE1.2: now also K5.4; no longer K5.7
- net at R100.1: now also U30.1
- net at R105.1: now also U16.5
- net at R106.1, U32.16 (A1): now also U16.11
- net at D15.2 (A): now also K7.1, U26.15; no longer K7.8
- net at D14.2 (A): now also K6.1, U30.15; no longer K6.8
- net at D13.2 (A): now also K3.1, U30.14; no longer K3.8
- net at R98.1: now also U26.1
- net at R107.1: now also U16.4
- net at R108.1, U32.1 (A0): now also U16.14
- net at K7.4: now also R110_RANGE1.2
- net at R110.1, U32.2 (ENABLE): now also U16.15
- net at K3.4: now also R108_RANGE1.2
- net at R101.1: now also U30.4
- net at R109.1: now also U16.1
- net at R104.1: now also U26.5; no longer U30.1
- net at D11.2 (A): now also K1.1, U26.14; no longer K1.8
- net at K6.4: now also R109_RANGE1.2
- new net: D8.2 (A), K2.1, U26.11
- new net: D10.2 (A), K5.1, U30.10
- now unconnected: K2.8, K5.8

Commit message: corrected kicad
Parts:
- R100, R101, R102, R103, R104, R98, R99: value 1k -> 150
Connections:
- net DAC_I_SENSE_+: now also K1.8, K2.8, K3.8, K4.8, K5.8, K6.8, K7.8; no longer K1.6, K2.6, K3.6, K4.6, K5.6, K6.6, K7.6
- net GNDA: no longer U16.7, U16.8, U26.7, U26.8
- net GNDD: now also U16.7, U16.8, U26.7, U26.8; no longer U30.7
Other:
- moved on the sheet: C182

Commit message: pcb 90%
Parts:
- added C59: 100nF, Capacitor_SMD:C_0805_2012Metric_Pad1.18x1.45mm_HandSolder, symbol Device:C_Small
Connections:
- net +12V_FILTERED: now also C59.2
- net GNDA: now also C59.1
Changed lines of the file:
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@@
 	)
 	(junction
+		(at 308.61 22.86)
+		(diameter 0)
+		(color 0 0 0 0)
+	)
+	(junction
 		(at 123.19 252.73)
 		(diameter 0)
@@
 	(wire
 		(pts
-			(xy 308.61 21.59) (xy 308.61 24.13)
+			(xy 308.61 21.59) (xy 308.61 22.86)
 		)
 		(stroke
@@
 	(wire
 		(pts
+			(xy 295.91 22.86) (xy 295.91 25.4)
+		)
+		(stroke
+			(width 0)
+			(type default)
+		)
+	)
+	(wire
+		(pts
 			(xy 137.16 177.8) (xy 68.58 177.8)
 		)
@@
 	(wire
 		(pts
+			(xy 304.8 22.86) (xy 308.61 22.86)
+		)
+		(stroke
+			(width 0)
+			(type default)
+		)
+	)
+	(wire
+		(pts
 			(xy 115.57 60.96) (xy 118.11 60.96)
 		)
@@
 	(wire
 		(pts
+			(xy 299.72 22.86) (xy 295.91 22.86)
+		)
+		(stroke
+			(width 0)
+			(type default)
+		)
+	)
+	(wire
+		(pts
 			(xy 168.91 157.48) (xy 168.91 160.02)
 		)
@@
 	(wire
 		(pts
+			(xy 308.61 22.86) (xy 308.61 24.13)
+		)
+		(stroke
+			(width 0)
+			(type default)
+		)
+	)
+	(wire
+		(pts
 			(xy 326.39 76.2) (xy 328.93 76.2)
 		)
@@
 	(symbol
 		(lib_id "power:GNDA")
+		(at 295.91 25.4 0)
+		(unit 1)
+		(exclude_from_sim no)
+		(in_bom yes)
+		(on_board yes)
+		(dnp no)
+		(property "Reference" "#PWR0134"
+			(at 295.91 31.75 0)
+			(effects
+				(font
+					(size 1.27 1.27)
+				)
+				(hide yes)
+			)
+		)
+		(property "Value" "GNDA"
+			(at 298.958 28.702 0)
+			(effects
+				(font
+					(size 1.27 1.27)
+				)
+			)
+		)
+		(property "Footprint" ""
+			(at 295.91 25.4 0)
+			(effects
+				(font
+					(size 1.27 1.27)
+				)
+				(hide yes)
+			)
+		)
+		(property "Datasheet" ""
+			(at 295.91 25.4 0)
+			(effects
+				(font
+					(size 1.27 1.27)
+				)
+				(hide yes)
+			)
+		)
+		(property "Description" "Power symbol creates a global label with name \"GNDA\" , analog ground"
+			(at 295.91 25.4 0)
+			(effects
+				(font
+					(size 1.27 1.27)
+				)
+				(hide yes)
+			)
+		)
+		(pin "1"
+		)
+		(instances
+			(project "ImpedanceAnalyzer"
+				(path "/08568624-f051-402a-adf3-1b03c2a769ee/83ca792e-0114-4481-9083-ddb809f73b86"
+					(reference "#PWR0134")
+					(unit 1)
+				)
+			)
+		)
+	)
+	(symbol
+		(lib_id "power:GNDA")
 		(at 124.46 137.16 0)
 		(unit 1)
@@
 					(unit 1)
 				)
+			)
+		)
+	)
+	(symbol
+		(lib_id "Device:C_Small")
+		(at 302.26 22.86 90)
+		(unit 1)
+		(exclude_from_sim no)
+		(in_bom yes)
+		(on_board yes)
+		(dnp no)
+		(property "Reference" "C59"
+			(at 300.99 17.78 0)
+			(effects
+				(font
+					(size 1.27 1.27)
+				)
+			)
+		)
+		(property "Value" "100nF"
+			(at 303.53 17.78 0)
+			(effects
+				(font
+					(size 1.27 1.27)
+				)
+			)
+		)
+		(property "Footprint" "Capacitor_SMD:C_0805_2012Metric_Pad1.18x1.45mm_HandSolder"
+			(at 302.26 22.86 0)
+			(effects
+				(font
+					(size 1.27 1.27)
+				)
+				(hide yes)
+			)
+		)
+		(property "Datasheet" "~"
+			(at 302.26 22.86 0)
+			(effects
+				(font
+					(size 1.27 1.27)
+				)
+				(hide yes)
+			)
+		)
+		(property "Description" "Unpolarized capacitor, small symbol"
+			(at 302.26 22.86 0)
+			(effects
+				(font
+					(size 1.27 1.27)
+				)
+				(hide yes)
+			)
+		)
+		(pin "2"
+		)
+		(pin "1"
+		)
+		(instances
+			(project "ImpedanceAnalyzer"
+				(path "/08568624-f051-402a-adf3-1b03c2a769ee/83ca792e-0114-4481-9083-ddb809f73b86"
+					(reference "C59")
+					(unit 1)
+				)
