File: PCB/ImpedanceAnalyzer/Supply.kicad_sch (KiCad schematic)
At the start: 0 parts

Commit message: schematic v1
Parts:
- added C147, C150, C152, C154, C155, C158, C160: 220uF, symbol Device:C_Polarized_Small
- added C148, C149, C151, C153, C156, C157, C159: 100nF, symbol Device:C_Small
- added C15, C16: 22uF, symbol Device:C_Polarized_Small
- added C17, C20, C21, C32, C42, C43, C44, C45, C46, C47: 510uF, symbol Device:C_Polarized_Small
- added D1, D2, D3, D4, D5, D6, D7: LED_RED, symbol Device:LED_Small
- added GND_LINK1: 0R, symbol Device:R_US
- added L1, L2: 1mH, symbol Device:L_Small
- added R32, R33: 1R1, symbol Device:R_Small
- added R79, R84: 1k, symbol Device:R_Small
- added R80, R83: 330R, symbol Device:R_Small
- added R81, R85: 390R, symbol Device:R_Small
- added R82: 150R, symbol Device:R_Small
- added U18: LM7812_TO220, Package_TO_SOT_THT:TO-220-3_Vertical, symbol Regulator_Linear:LM7812_TO220
- added U19: LM7912_TO220, Package_TO_SOT_THT:TO-220-3_Vertical, symbol Regulator_Linear:LM7912_TO220
- added U20: LM7806_TO220, Package_TO_SOT_THT:TO-220-3_Vertical, symbol Regulator_Linear:LM7806_TO220
- added U21: LT1086-3.3, symbol Regulator_Linear:LT1086-3.3
- added U22: LM7805_TO220, Package_TO_SOT_THT:TO-220-3_Vertical, symbol Regulator_Linear:LM7805_TO220
- added U23: LM7905_TO220, Package_TO_SOT_THT:TO-220-3_Vertical, symbol Regulator_Linear:LM7905_TO220
- added U24: LM7906_TO220, Package_TO_SOT_THT:TO-220-3_Vertical, symbol Regulator_Linear:LM7906_TO220
Connections:
- new net: D1.2 (A), R79.2
- new net: D6.1 (K), R84.2
- new net: D2.2 (A), R80.2
- new net: D4.2 (A), R82.2
- new net: D5.1 (K), R83.2
- new net: C147.1, C15.1, C17.1, C21.1, C42.1, C44.1, C46.1, L1.1, U18.1 (VI)
- new net: C17.2, C21.2, C42.2, C44.2, C46.2, R32.2
- new net: C155.2, C16.1, C20.1, C32.1, C43.1, C45.1, C47.1, L2.1, U19.2 (VI)
- new net: C20.2, C32.2, C43.2, C45.2, C47.2, R33.2
- new net: D7.1 (K), R85.2
- new net: D3.2 (A), R81.2
- new net +12V_FILTERED: C148.1, C149.1, C151.1, C153.1, R79.1, U18.3 (VO), U20.1 (VI), U21.3 (VI), U22.1 (VI)
- new net +15V_MW: L1.2
- new net +3V3_REG: C154.1, R82.1, U21.2 (VO)
- new net +5V_REG: C150.1, D7.2 (A), R80.1, U22.3 (VO), U24.1 (GND)
- new net +6V_REG: C152.1, R81.1, U20.3 (VO)
- new net -12V_FILTERED: C156.1, C159.1, R84.1, U19.3 (VO), U23.2 (VI)
- new net -15V_MW: L2.2
- new net -1V_REG: C158.2, R85.1, U24.3 (VO)
- new net -5V_REG: C157.1, C160.2, R83.1, U23.3 (VO), U24.2 (VI)
- new net GNDA: C147.2, C148.2, C149.2, C15.2, C150.2, C151.2, C152.2, C155.1, C156.2, C157.2, C158.1, C159.2, C16.2, C160.1, D1.1 (K), D2.1 (K), D3.1 (K), D4.1 (K), D5.2 (A), D6.2 (A), GND_LINK1.1, R32.1, R33.1, U18.2 (GND), U19.1 (GND), U20.2 (GND), U22.2 (GND), U23.1 (GND)
- new net GNDD: C153.2, C154.2, U21.1 (GND)
- new net GND_MW: GND_LINK1.2
Other:
- note added: "ANALOG/MEAN WELL GROUND LINK"

Commit message: ready for pcb
Parts:
- removed C147, C150, C152, C154, C155, C158, C160: 220uF, symbol Device:C_Polarized_Small
- added C147, C150, C152, C154, C155, C158, C160: 1uF, Capacitor_SMD:C_0805_2012Metric_Pad1.18x1.45mm_HandSolder, symbol Device:C_Small
- C148, C149, C151, C153, C156, C157, C159: footprint (none) -> Capacitor_SMD:C_0805_2012Metric_Pad1.18x1.45mm_HandSolder
- C15, C16: footprint (none) -> Capacitor_THT:CP_Radial_D6.3mm_P2.50mm
- C17, C20, C21, C32, C42, C43, C44, C45, C46, C47: footprint (none) -> Capacitor_THT:CP_Radial_D10.0mm_P5.00mm
- D1, D2, D3, D4, D5, D6, D7: footprint (none) -> LED_THT:LED_D2.0mm_W4.0mm_H2.8mm_FlatTop
- GND_LINK1: footprint (none) -> JRIX Resistor SMD:Resistor SMD - 2818
- L1, L2: footprint (none) -> JRIX Inductor THT Footprints:INDRD1000W100D1800H2550 - AIUR-15-102K
- R32, R33, R79, R80, R81, R82, R83, R84, R85: footprint (none) -> Resistor_THT:R_Axial_DIN0207_L6.3mm_D2.5mm_P10.16mm_Horizontal
- U21: footprint (none) -> Package_TO_SOT_THT:TO-220-3_Vertical
Connections:
- net +3V3_REG: now also C154.1
- net +5V_REG: now also C150.1
- net +6V_REG: now also C152.1
- net -1V_REG: now also C158.1
- net -5V_REG: now also C160.1
- net GNDA: now also C147.2, C150.2, C152.2, C155.2, C158.2, C160.2
- net GNDD: now also C154.2
- net at C15.1, C17.1, C21.1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: now also C147.1
- net at C16.1, C20.1, C32.1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: now also C155.1
Other:
- note added: "LEDs are L424IDT"

Commit message: corrected kicad
Parts:
- added C211: 100nF, Capacitor_SMD:C_0805_2012Metric_Pad1.18x1.45mm_HandSolder, symbol Device:C_Small
- added C212: 10uF, Capacitor_SMD:C_1210_3225Metric, symbol Device:C_Small
- added D19: LED_RED, LED_THT:LED_D2.0mm_W4.0mm_H2.8mm_FlatTop, symbol Device:LED_Small
- added R31, R34: 150R, Resistor_THT:R_Axial_DIN0207_L6.3mm_D2.5mm_P10.16mm_Horizontal, symbol Device:R_Small
- added U28: LD1117S25TR_SOT223, Package_TO_SOT_SMD:SOT-223-3_TabPin2, symbol Regulator_Linear:LD1117S25TR_SOT223
Connections:
- net +12V_FILTERED: no longer C153.1, U21.3 (VI)
- net GNDA: now also C211.2, C212.2, D19.1 (K), U28.1 (GND); no longer D4.1 (K)
- net GNDD: now also D4.1 (K)
- new net: D19.2 (A), R31.2, R34.2
- new net: C211.1, U28.3 (VI)
- new net +2V5_REG: C212.1, R31.1, R34.1, U28.2 (VO)
- new net +5V_MW: C153.1, U21.3 (VI)
Other:
- moved on the sheet: C153, C154, C155, C156, C157, C158, C159, C16, C160, C20, C21, C32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

Commit message: pcb 90%
Connections:
- net +5V_REG: now also C211.1, U28.3 (VI)
- net GNDA: now also C155.1, C16.1; no longer C155.2, C16.2
- net at C20.1, C32.1, C43.1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: now also R33.2; no longer C155.1, C16.1, L2.1, U19.2 (VI)
- net at C20.2, C32.2, C43.2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: now also C155.2, C16.2, L2.1, U19.2 (VI); no longer R33.2
Other:
- moved on the sheet: C155, C16, C20, C32, C43, C45, C47
Changed lines of the file:
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@@
 	)
 	(junction
+		(at 48.26 93.98)
+		(diameter 0)
+		(color 0 0 0 0)
+	)
+	(junction
 		(at 62.23 64.77)
 		(diameter 0)
@@
 	)
 	(junction
+		(at 115.57 104.14)
+		(diameter 0)
+		(color 0 0 0 0)
+	)
+	(junction
 		(at 71.12 64.77)
 		(diameter 0)
@@
 	(wire
 		(pts
-			(xy 48.26 35.56) (xy 48.26 160.02)
+			(xy 48.26 35.56) (xy 48.26 93.98)
 		)
 		(stroke
@@
 	(wire
 		(pts
+			(xy 48.26 93.98) (xy 48.26 160.02)
+		)
+		(stroke
+			(width 0)
+			(type default)
+		)
+	)
+	(wire
+		(pts
 			(xy 66.04 179.07) (xy 66.04 180.34)
 		)
@@
 	(wire
 		(pts
+			(xy 115.57 104.14) (xy 115.57 93.98)
+		)
+		(stroke
+			(width 0)
+			(type default)
+		)
+	)
+	(wire
+		(pts
 			(xy 66.04 171.45) (xy 66.04 173.99)
 		)
@@
 	(wire
 		(pts
+			(xy 115.57 93.98) (xy 48.26 93.98)
+		)
+		(stroke
+			(width 0)
+			(type default)
+		)
+	)
+	(wire
+		(pts
 			(xy 182.88 87.63) (xy 172.72 87.63)
 		)
@@
 	(symbol
 		(lib_id "Device:C_Polarized_Small")
-		(at 217.17 130.81 0)
+		(at 217.17 130.81 180)
 		(unit 1)
 		(exclude_from_sim no)
@@
 		(dnp no)
 		(property "Reference" "C32"
-			(at 218.948 129.54 0)
+			(at 215.392 132.08 0)
 			(effects
 				(font
@@
 		)
 		(property "Value" "510uF"
-			(at 218.948 132.08 0)
+			(at 215.392 129.54 0)
 			(effects
 				(font
@@
 	(symbol
 		(lib_id "Device:C_Polarized_Small")
-		(at 198.12 130.81 0)
+		(at 198.12 130.81 180)
 		(unit 1)
 		(exclude_from_sim no)
@@
 		(dnp no)
 		(property "Reference" "C16"
-			(at 199.898 129.54 0)
+			(at 196.342 132.08 0)
 			(effects
 				(font
@@
 		)
 		(property "Value" "22uF"
-			(at 199.898 132.08 0)
+			(at 196.342 129.54 0)
 			(effects
 				(font
@@
 	(symbol
 		(lib_id "Device:C_Polarized_Small")
-		(at 250.19 130.81 0)
+		(at 250.19 130.81 180)
 		(unit 1)
 		(exclude_from_sim no)
@@
 		(fields_autoplaced yes)
 		(property "Reference" "C47"
-			(at 252.73 128.9938 0)
+			(at 252.73 130.086 0)
 			(effects
 				(font
 					(size 1.27 1.27)
 				)
-				(justify left)
+				(justify right)
 			)
 		)
 		(property "Value" "510uF"
-			(at 252.73 131.5338 0)
+			(at 252.73 132.626 0)
 			(effects
 				(font
 					(size 1.27 1.27)
 				)
-				(justify left)
+				(justify right)
 			)
 		)
@@
 	(symbol
 		(lib_id "Device:C_Small")
-		(at 186.69 130.81 0)
+		(at 186.69 130.81 180)
 		(unit 1)
 		(exclude_from_sim no)
@@
 		(dnp no)
 		(property "Reference" "C155"
-			(at 189.23 129.5462 0)
+			(at 184.15 132.0738 0)
 			(effects
 				(font
@@
 		)
 		(property "Value" "1uF"
-			(at 188.976 132.08 0)
+			(at 184.404 129.54 0)
 			(effects
 				(font
@@
 	(symbol
 		(lib_id "Device:C_Polarized_Small")
-		(at 207.01 130.81 0)
+		(at 207.01 130.81 180)
 		(unit 1)
 		(exclude_from_sim no)
@@
 		(dnp no)
 		(property "Reference" "C20"
-			(at 208.788 129.794 0)
+			(at 205.232 131.826 0)
 			(effects
 				(font
@@
 		)
 		(property "Value" "510uF"
-			(at 208.788 132.334 0)
+			(at 205.232 129.286 0)
 			(effects
 				(font
@@
 	(symbol
 		(lib_id "Device:C_Polarized_Small")
-		(at 238.76 130.81 0)
+		(at 238.76 130.81 180)
 		(unit 1)
 		(exclude_from_sim no)
@@
 		(dnp no)
 		(property "Reference" "C45"
-			(at 241.3 128.9938 0)
+			(at 236.22 132.6262 0)
 			(effects
 				(font
@@
 		)
 		(property "Value" "510uF"
-			(at 241.3 131.5338 0)
+			(at 236.22 130.0862 0)
 			(effects
 				(font
@@
 	(symbol
 		(lib_id "Device:C_Polarized_Small")
-		(at 227.33 130.81 0)
+		(at 227.33 130.81 180)
 		(unit 1)
 		(exclude_from_sim no)
@@
 		(dnp no)
 		(property "Reference" "C43"
-			(at 229.616 129.54 0)
+			(at 225.044 132.08 0)
 			(effects
 				(font
@@
 		)
 		(property "Value" "510uF"
-			(at 229.616 132.08 0)
+			(at 225.044 129.54 0)
 			(effects
 				(font
