File: PCB/ImpedanceAnalyzer/digital.kicad_sch (KiCad schematic)
At the start: 22 parts, among them M1 Artix_7_35T_CMOD_A7, U10 NUCLEO-F446RE, U15 74HC14, U27 74HC595

Commit message: ready for pcb
Parts:
- removed C134, C135, C136, C138, C139, C140: 220uF, symbol Device:C_Polarized_Small
- added C134, C135, C136, C138, C139, C140: 1uF, Capacitor_SMD:C_0805_2012Metric_Pad1.18x1.45mm_HandSolder, symbol Device:C_Small
- C130, C131, C141, C143, C146, C173: footprint (none) -> Capacitor_SMD:C_0805_2012Metric_Pad1.18x1.45mm_HandSolder
- C132, C133, C144, C145: value 220uF -> 470uF; footprint (none) -> Capacitor_THT:CP_Radial_D10.0mm_P5.00mm
- C137, C142: footprint (none) -> Capacitor_THT:C_Disc_D3.4mm_W2.1mm_P2.50mm
- M1: footprint (none) -> JRIX FPGA Footprints:CMOD A7 Module
- U10: footprint NUCLEO-F446RE:MODULE_NUCLEO-F446RE -> JRIX STM32 Development Boards Footprint:MODULE_NUCLEO-F446RE
- U15: footprint (none) -> Package_DIP:DIP-14_W7.62mm
- U27: footprint (none) -> Package_DIP:DIP-16_W7.62mm
Connections:
- net +3V3_REG: now also C138.2, C139.2, C140.2
- net +5V_MW_REG: now also C134.1, C135.1, C136.1
- net GNDD: now also C134.2, C135.2, C136.2, C138.1, C139.1, C140.1

Commit message: corrected kicad
Connections:
- net +3V3_REG: now also U27.10 (~{SRCLR})
- net +5V_MW_REG: no longer U27.10 (~{SRCLR})
- net ADC2MISO: now also M1.5 (PIO5); no longer M1.4 (PIO4)
- net ADC2SCK: now also M1.4 (PIO4); no longer M1.3 (PIO3)
- net ADCCNV: now also M1.3 (PIO3); no longer M1.5 (PIO5)
Changed lines of the file:
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@@
 	(wire
 		(pts
-			(xy 48.26 87.63) (xy 52.07 87.63)
-		)
-		(stroke
-			(width 0)
-			(type default)
-		)
-	)
-	(wire
-		(pts
 			(xy 74.93 80.01) (xy 100.33 80.01)
 		)
@@
 	(wire
 		(pts
-			(xy 48.26 82.55) (xy 52.07 82.55)
-		)
-		(stroke
-			(width 0)
-			(type default)
-		)
-	)
-	(wire
-		(pts
 			(xy 217.17 96.52) (xy 217.17 95.25)
 		)
@@
 	(wire
 		(pts
-			(xy 48.26 85.09) (xy 52.07 85.09)
-		)
-		(stroke
-			(width 0)
-			(type default)
-		)
-	)
-	(wire
-		(pts
 			(xy 29.21 35.56) (xy 44.45 35.56)
 		)
@@
 	(wire
 		(pts
-			(xy 92.71 26.67) (xy 101.6 26.67)
+			(xy 48.26 82.55) (xy 52.07 82.55)
+		)
+		(stroke
+			(width 0)
+			(type default)
+		)
+	)
+	(wire
+		(pts
+			(xy 92.71 26.67) (xy 105.41 26.67)
 		)
 		(stroke
@@
 	(wire
 		(pts
-			(xy 101.6 26.67) (xy 101.6 27.94)
+			(xy 105.41 26.67) (xy 105.41 27.94)
 		)
 		(stroke
@@
 	(wire
 		(pts
+			(xy 48.26 85.09) (xy 52.07 85.09)
+		)
+		(stroke
+			(width 0)
+			(type default)
+		)
+	)
+	(wire
+		(pts
 			(xy 209.55 199.39) (xy 215.9 199.39)
 		)
@@
 	(wire
 		(pts
+			(xy 48.26 87.63) (xy 52.07 87.63)
+		)
+		(stroke
+			(width 0)
+			(type default)
+		)
+	)
+	(wire
+		(pts
 			(xy 233.68 96.52) (xy 233.68 95.25)
 		)
@@
 		)
 	)
-	(label "+5V"
-		(at 78.74 187.96 0)
-		(fields_autoplaced yes)
-		(effects
-			(font
-				(size 1.27 1.27)
-			)
-			(justify left bottom)
-		)
-	)
 	(label "DB15"
 		(at 215.9 199.39 180)
@@
 		)
 	)
+	(label "+3V3"
+		(at 78.74 187.96 0)
+		(fields_autoplaced yes)
+		(effects
+			(font
+				(size 1.27 1.27)
+			)
+			(justify left bottom)
+		)
+	)
 	(label "DB3"
 		(at 168.91 224.79 0)
@@
 	(hierarchical_label "ADCCNV"
 		(shape output)
-		(at 48.26 87.63 180)
+		(at 48.26 82.55 180)
 		(fields_autoplaced yes)
 		(effects
@@
 	(hierarchical_label "ADC2MISO"
 		(shape input)
-		(at 48.26 85.09 180)
+		(at 48.26 87.63 180)
 		(fields_autoplaced yes)
 		(effects
@@
 	(hierarchical_label "ADC2SCK"
 		(shape output)
-		(at 48.26 82.55 180)
+		(at 48.26 85.09 180)
 		(fields_autoplaced yes)
 		(effects
@@
 	(symbol
 		(lib_id "power:GNDD")
-		(at 101.6 27.94 0)
+		(at 105.41 27.94 0)
 		(unit 1)
 		(exclude_from_sim no)
@@
 		(fields_autoplaced yes)
 		(property "Reference" "#PWR050"
-			(at 101.6 34.29 0)
+			(at 105.41 34.29 0)
 			(effects
 				(font
@@
 		)
 		(property "Value" "GNDD"
-			(at 101.6 31.75 0)
+			(at 105.41 31.75 0)
 			(effects
 				(font
@@
 		)
 		(property "Footprint" ""
-			(at 101.6 27.94 0)
+			(at 105.41 27.94 0)
 			(effects
 				(font
@@
 		)
 		(property "Datasheet" ""
-			(at 101.6 27.94 0)
+			(at 105.41 27.94 0)
 			(effects
 				(font
@@
 		)
 		(property "Description" "Power symbol creates a global label with name \"GNDD\" , digital ground"
-			(at 101.6 27.94 0)
+			(at 105.41 27.94 0)
 			(effects
 				(font
@@
 		(on_board yes)
 		(dnp no)
-		(fields_autoplaced yes)
 		(property "Reference" "C142"
-			(at 41.91 31.7438 0)
+			(at 51.562 30.988 0)
 			(effects
 				(font
@@
 		)
 		(property "Value" "100pF"
-			(at 41.91 29.2038 0)
+			(at 51.562 28.448 0)
 			(effects
 				(font
@@
 		(on_board yes)
 		(dnp no)
-		(fields_autoplaced yes)
 		(property "Reference" "C141"
-			(at 52.07 31.7438 0)
+			(at 61.722 30.988 0)
 			(effects
 				(font
@@
 		)
 		(property "Value" "100nF"
-			(at 52.07 29.2038 0)
+			(at 61.722 28.448 0)
 			(effects
 				(font

Commit message: pcb 90%
Connections:
- net ADC1MISO: now also M1.5 (PIO5); no longer M1.2 (PIO2)
- net ADC1SCK: now also M1.4 (PIO4); no longer M1.1 (PIO1)
- net ADC2MISO: now also M1.2 (PIO2); no longer M1.5 (PIO5)
- net ADC2SCK: now also M1.1 (PIO1); no longer M1.4 (PIO4)
- net DACB12: now also M1.29 (PIO29); no longer M1.26 (PIO26)
- net DACB13: now also M1.28 (PIO28); no longer M1.27 (PIO27)
- net DACB14: now also M1.26 (PIO26); no longer M1.28 (PIO28)
- net DACB15: now also M1.27 (PIO27); no longer M1.29 (PIO29)
Changed lines of the file:
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@@
 		)
 	)
-	(hierarchical_label "ADC1SCK"
+	(hierarchical_label "DACB2"
+		(shape output)
+		(at 49.53 105.41 180)
+		(fields_autoplaced yes)
+		(effects
+			(font
+				(size 1.27 1.27)
+			)
+			(justify right)
+		)
+	)
+	(hierarchical_label "DACB10"
+		(shape output)
+		(at 49.53 130.81 180)
+		(fields_autoplaced yes)
+		(effects
+			(font
+				(size 1.27 1.27)
+			)
+			(justify right)
+		)
+	)
+	(hierarchical_label "ADC2MISO"
+		(shape input)
+		(at 48.26 80.01 180)
+		(fields_autoplaced yes)
+		(effects
+			(font
+				(size 1.27 1.27)
+			)
+			(justify right)
+		)
+	)
+	(hierarchical_label "DACB12"
+		(shape output)
+		(at 77.47 125.73 0)
+		(fields_autoplaced yes)
+		(effects
+			(font
+				(size 1.27 1.27)
+			)
+			(justify left)
+		)
+	)
+	(hierarchical_label "ADC2SCK"
 		(shape output)
 		(at 48.26 77.47 180)
@@
 		)
 	)
-	(hierarchical_label "DACB2"
-		(shape output)
-		(at 49.53 105.41 180)
-		(fields_autoplaced yes)
-		(effects
-			(font
-				(size 1.27 1.27)
-			)
-			(justify right)
-		)
-	)
-	(hierarchical_label "DACB10"
-		(shape output)
-		(at 49.53 130.81 180)
-		(fields_autoplaced yes)
-		(effects
-			(font
-				(size 1.27 1.27)
-			)
-			(justify right)
-		)
-	)
 	(hierarchical_label "DACB11"
 		(shape output)
@@
 			)
 			(justify right)
-		)
-	)
-	(hierarchical_label "DACB15"
-		(shape output)
-		(at 77.47 125.73 0)
-		(fields_autoplaced yes)
-		(effects
-			(font
-				(size 1.27 1.27)
-			)
-			(justify left)
 		)
 	)
@@
 		)
 	)
+	(hierarchical_label "ADC1MISO"
+		(shape input)
+		(at 48.26 87.63 180)
+		(fields_autoplaced yes)
+		(effects
+			(font
+				(size 1.27 1.27)
+			)
+			(justify right)
+		)
+	)
 	(hierarchical_label "DACCLK"
 		(shape output)
@@
 		)
 	)
+	(hierarchical_label "DACB13"
+		(shape output)
+		(at 77.47 128.27 0)
+		(fields_autoplaced yes)
+		(effects
+			(font
+				(size 1.27 1.27)
+			)
+			(justify left)
+		)
+	)
+	(hierarchical_label "DACB6"
+		(shape output)
+		(at 49.53 120.65 180)
+		(fields_autoplaced yes)
+		(effects
+			(font
+				(size 1.27 1.27)
+			)
+			(justify right)
+		)
+	)
+	(hierarchical_label "I_PGA_A0"
+		(shape output)
+		(at 170.18 245.11 180)
+		(fields_autoplaced yes)
+		(effects
+			(font
+				(size 1.27 1.27)
+			)
+			(justify right)
+		)
+	)
+	(hierarchical_label "RANGEB3"
+		(shape output)
+		(at 50.8 187.96 180)
+		(fields_autoplaced yes)
+		(effects
+			(font
+				(size 1.27 1.27)
+			)
+			(justify right)
+		)
+	)
+	(hierarchical_label "I_PGA_A1"
+		(shape output)
+		(at 170.18 247.65 180)
+		(fields_autoplaced yes)
+		(effects
+			(font
+				(size 1.27 1.27)
+			)
+			(justify right)
+		)
+	)
+	(hierarchical_label "RANGEB0"
+		(shape output)
+		(at 50.8 180.34 180)
+		(fields_autoplaced yes)
+		(effects
+			(font
+				(size 1.27 1.27)
+			)
+			(justify right)
+		)
+	)
+	(hierarchical_label "DACB8"
+		(shape output)
+		(at 49.53 125.73 180)
+		(fields_autoplaced yes)
+		(effects
+			(font
+				(size 1.27 1.27)
+			)
+			(justify right)
+		)
+	)
 	(hierarchical_label "DACB14"
 		(shape output)
-		(at 77.47 128.27 0)
+		(at 77.47 133.35 0)
 		(fields_autoplaced yes)
 		(effects
@@
 			)
 			(justify left)
-		)
-	)
-	(hierarchical_label "DACB6"
-		(shape output)
-		(at 49.53 120.65 180)
-		(fields_autoplaced yes)
-		(effects
-			(font
-				(size 1.27 1.27)
-			)
-			(justify right)
-		)
-	)
-	(hierarchical_label "I_PGA_A0"
-		(shape output)
-		(at 170.18 245.11 180)
-		(fields_autoplaced yes)
-		(effects
-			(font
-				(size 1.27 1.27)
-			)
-			(justify right)
-		)
-	)
-	(hierarchical_label "RANGEB3"
-		(shape output)
-		(at 50.8 187.96 180)
-		(fields_autoplaced yes)
-		(effects
-			(font
-				(size 1.27 1.27)
-			)
-			(justify right)
-		)
-	)
-	(hierarchical_label "I_PGA_A1"
-		(shape output)
-		(at 170.18 247.65 180)
-		(fields_autoplaced yes)
-		(effects
-			(font
-				(size 1.27 1.27)
-			)
-			(justify right)
-		)
-	)
-	(hierarchical_label "ADC1MISO"
-		(shape input)
-		(at 48.26 80.01 180)
-		(fields_autoplaced yes)
-		(effects
-			(font
-				(size 1.27 1.27)
-			)
-			(justify right)
-		)
-	)
-	(hierarchical_label "RANGEB0"
-		(shape output)
-		(at 50.8 180.34 180)
-		(fields_autoplaced yes)
-		(effects
-			(font
-				(size 1.27 1.27)
-			)
-			(justify right)
-		)
-	)
-	(hierarchical_label "ADC2MISO"
-		(shape input)
-		(at 48.26 87.63 180)
-		(fields_autoplaced yes)
-		(effects
-			(font
-				(size 1.27 1.27)
-			)
-			(justify right)
-		)
-	)
-	(hierarchical_label "DACB8"
-		(shape output)
-		(at 49.53 125.73 180)
-		(fields_autoplaced yes)
-		(effects
-			(font
-				(size 1.27 1.27)
-			)
-			(justify right)
 		)
 	)
@@
 		)
 	)
-	(hierarchical_label "ADC2SCK"
-		(shape output)
-		(at 48.26 85.09 180)
-		(fields_autoplaced yes)
-		(effects
-			(font
-				(size 1.27 1.27)
-			)
-			(justify right)
-		)
-	)
-	(hierarchical_label "DACB13"
-		(shape output)
-		(at 77.47 130.81 0)
-		(fields_autoplaced yes)
-		(effects
-			(font
-				(size 1.27 1.27)
-			)
-			(justify left)
-		)
-	)
 	(hierarchical_label "+3V3_REG"
 		(shape input)
@@
 		)
 	)
+	(hierarchical_label "DACB15"
+		(shape output)
+		(at 77.47 130.81 0)
+		(fields_autoplaced yes)
+		(effects
+			(font
+				(size 1.27 1.27)
+			)
+			(justify left)
+		)
+	)
+	(hierarchical_label "ADC1SCK"
+		(shape output)
+		(at 48.26 85.09 180)
+		(fields_autoplaced yes)
+		(effects
+			(font
+				(size 1.27 1.27)
+			)
+			(justify right)
+		)
+	)
 	(hierarchical_label "RANGEB4"
 		(shape output)
@@
 		)
 	)
-	(hierarchical_label "DACB12"
-		(shape output)
-		(at 77.47 133.35 0)
-		(fields_autoplaced yes)
-		(effects
-			(font
-				(size 1.27 1.27)
-			)
-			(justify left)
-		)
-	)
