File: PCB/ImpedanceAnalyzer/ImpedanceAnalyzer.kicad_pcb (KiCad board)
At the start: 4 copper layers, 414 parts, among them J1 63849-1, J10 63849-1, J2 63849-1, J3 63849-1, J5 Conn_01x04, J6 DUT_H_POT, J7 DUT_L_POT, J8 DUT_H_CUR, J9 DUT_L_CUR, K1 RY-12W-K, K2 RY-12W-K, K3 RY-12W-K, K4 RY-12W-K, K5 RY-12W-K, K6 RY-12W-K, K7 RY-12W-K, M1 Artix_7_35T_CMOD_A7, Q1 BC547, Q2 BC557, Q3 BC547, Q4 BC557, U1 LTC2311, U10 NUCLEO-F446RE, U11 OPA4830, U12 REF02Z, U13 OPA2277-EP, U14 OPA4830, U15 74HC14, U16 ILQ1, U17 OPA4830, U18 LM7812_TO220, U19 LM7912_TO220, U2 LTC2311, U20 LM7806_TO220, U21 LT1086-3.3, U22 LM7805_TO220, U23 LM7905_TO220, U24 LM7906_TO220, U25 PGA855, U26 ILQ1, U27 74HC595, U28 LD1117S25TR_SOT223, U3 LT1819, U30 ILQ1, U31 ILQ1, U32 MUX-24, U33 ILQ1, U34 AD8032, U35 PGA855, U4 LT1819, U5 OPA350, U6 LTC1668CG, U7 OPA350, U8 OPA4830, U9 OPA4830

Commit message: pcb 90%
Parts:
- removed C60, C67, C68: 100pF, Capacitor_THT:C_Disc_D3.4mm_W2.1mm_P2.50mm
- C10, C12, C131, C135, C136, C14, C143, C146, C178, C179, C18, C180, C181, C183, C184, C185, C23, C24, C25, C28, C48, C66, C89, C90, C91, C94: moved to B.Cu
- C29: value 470uF -> 100uF; footprint Capacitor_THT:CP_Radial_D10.0mm_P5.00mm -> Capacitor_SMD:C_1206_3216Metric_Pad1.33x1.80mm_HandSolder; moved to B.Cu
- C3, C4, C7, C88, C93: footprint Capacitor_THT:CP_Radial_D6.3mm_P2.50mm -> Capacitor_SMD:C_1206_3216Metric_Pad1.33x1.80mm_HandSolder; moved to B.Cu
- C59: value 100pF -> 100nF; footprint Capacitor_THT:C_Disc_D3.4mm_W2.1mm_P2.50mm -> Capacitor_SMD:C_0805_2012Metric_Pad1.18x1.45mm_HandSolder
- C86: value 100u -> 100uF; footprint Capacitor_THT:CP_Radial_D6.3mm_P2.50mm -> Capacitor_SMD:C_1206_3216Metric_Pad1.33x1.80mm_HandSolder; moved to B.Cu
- moved U16 522.2 mm to (314.7, 149.2), turned to -90 degrees
- moved U26 487.7 mm to (290.4, 149.3), turned to -90 degrees
- moved R109 483.5 mm to (314.7, 144.1), turned to 90 degrees
- moved R110 483.0 mm to (312.1, 160.5), turned to -90 degrees
- moved R108 480.6 mm to (308.6, 160.5), turned to 180 degrees
- moved R107 479.5 mm to (307.1, 144.1), turned to 90 degrees
- moved R106 478.7 mm to (303.5, 160.1)
- moved R105 477.7 mm to (304.5, 144.1), turned to 90 degrees
- moved R98 469.2 mm to (290.3, 144.1), turned to 90 degrees
- moved C173 468.9 mm to (322.4, 124.6), turned to 90 degrees
- moved R99 461.2 mm to (282.7, 144.1), turned to 90 degrees
- moved C138 456.1 mm to (310.4, 81.4), turned to -90 degrees
- moved C140 455.9 mm to (310.4, 86.0), turned to 90 degrees
- moved R104 454.2 mm to (280.3, 144.1), turned to 90 degrees
- moved U30 452.7 mm to (265.4, 149.3), turned to -90 degrees
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Connections:
- C10 pad 1: GNDD -> GNDA
- C102 pad 2: GNDD -> GNDA
- C103 pad 1: GNDD -> GNDA
- C104 pad 2: GNDD -> GNDA
- C105 pad 1: GNDD -> GNDA
- C106 pad 1: GNDD -> GNDA
- C107 pad 1: GNDD -> GNDA
- C11 pad 2: GNDD -> GNDA
- C110 pad 1: GNDD -> GNDA
- C111 pad 1: GNDD -> GNDA
- C114 pad 1: GNDD -> GNDA
- C115 pad 1: GNDD -> GNDA
- C118 pad 2: GNDD -> GNDA
- C119 pad 1: GNDD -> GNDA
- C12 pad 1: GNDD -> GNDA
- C120 pad 2: GNDD -> GNDA
- C121 pad 1: GNDD -> GNDA
- C122 pad 2: GNDD -> GNDA
- C123 pad 1: GNDD -> GNDA
- C124 pad 2: GNDD -> GNDA
- C125 pad 1: GNDD -> GNDA
- C126 pad 2: GNDD -> GNDA
- C127 pad 1: GNDD -> GNDA
- C128 pad 2: GNDD -> GNDA
- C129 pad 1: GNDD -> GNDA
- C13 pad 2: GNDD -> GNDA
- C130 pad 2: GNDD -> GNDA
- C131 pad 2: GNDD -> GNDA
- C132 pad 2: GNDD -> GNDA
- C133 pad 2: GNDD -> GNDA
- C134 pad 2: GNDD -> GNDA
- C135 pad 2: GNDD -> GNDA
- C136 pad 2: GNDD -> GNDA
- C137 pad 2: GNDD -> GNDA
- C138 pad 1: GNDD -> GNDA
- C139 pad 1: GNDD -> GNDA
- C14 pad 2: GNDD -> GNDA
- C140 pad 1: GNDD -> GNDA
- C141 pad 2: GNDD -> GNDA
- C142 pad 2: GNDD -> GNDA
- C143 pad 1: GNDD -> GNDA
- C144 pad 2: GNDD -> GNDA
- C145 pad 2: GNDD -> GNDA
- C146 pad 1: GNDD -> GNDA
- C147 pad 2: GNDD -> GNDA
- C148 pad 2: GNDD -> GNDA
- C149 pad 2: GNDD -> GNDA
- C15 pad 2: GNDD -> GNDA
- C150 pad 2: GNDD -> GNDA
- C151 pad 2: GNDD -> GNDA
- C152 pad 2: GNDD -> GNDA
- C153 pad 2: GNDD -> GNDA
- C154 pad 2: GNDD -> GNDA
- C155 pad 1: Net-(U19-VI) -> GNDA
- C155 pad 2: GNDD -> Net-(U19-VI)
- C156 pad 2: GNDD -> GNDA
- C157 pad 2: GNDD -> GNDA
- C158 pad 2: GNDD -> GNDA
- C159 pad 2: GNDD -> GNDA
- C16 pad 1: Net-(U19-VI) -> GNDA
- C16 pad 2: GNDD -> Net-(U19-VI)
- C160 pad 2: GNDD -> GNDA
- C161 pad 2: GNDD -> GNDA
- C162 pad 2: GNDD -> GNDA
- C163 pad 2: GNDD -> GNDA
- C164 pad 2: GNDD -> GNDA
- C165 pad 2: GNDD -> GNDA
- C166 pad 2: GNDD -> GNDA
- C167 pad 2: GNDD -> GNDA
- C168 pad 2: GNDD -> GNDA
- C169 pad 2: GNDD -> GNDA
- C170 pad 2: GNDD -> GNDA
- C171 pad 2: GNDD -> GNDA
- C172 pad 2: GNDD -> GNDA
- C173 pad 1: GNDD -> GNDA
- C174 pad 2: GNDD -> GNDA
- C175 pad 2: GNDD -> GNDA
- C176 pad 2: GNDD -> GNDA
- C177 pad 2: GNDD -> GNDA
- C178 pad 2: GNDD -> GNDA
- C179 pad 2: GNDD -> GNDA
- C18 pad 2: GNDD -> GNDA
- C180 pad 2: GNDD -> GNDA
- C181 pad 2: GNDD -> GNDA
- C182 pad 2: GNDD -> GNDA
- C183 pad 2: GNDD -> GNDA
- C184 pad 2: GNDD -> GNDA
- C185 pad 2: GNDD -> GNDA
- C186 pad 1: GNDD -> GNDA
- C187 pad 2: GNDD -> GNDA
- C188 pad 2: GNDD -> GNDA
- C189 pad 2: GNDD -> GNDA
- C19 pad 2: GNDD -> GNDA
- C190 pad 2: GNDD -> GNDA
- C191 pad 2: GNDD -> GNDA
- C192 pad 2: GNDD -> GNDA
- C193 pad 1: GNDD -> GNDA
- C194 pad 2: GNDD -> GNDA
- C195 pad 2: GNDD -> GNDA
- C196 pad 2: GNDD -> GNDA
- C197 pad 1: GNDD -> GNDA
- C198 pad 2: GNDD -> GNDA
- C20 pad 1: Net-(U19-VI) -> Net-(C20-Pad1)
- C20 pad 2: Net-(C20-Pad2) -> Net-(U19-VI)
- C203 pad 2: GNDD -> GNDA
- C204 pad 1: GNDD -> GNDA
- C205 pad 2: GNDD -> GNDA
- C206 pad 1: GNDD -> GNDA
- C211 pad 1: Net-(U28-VI) -> /ADC/+5V
- C211 pad 2: GNDD -> GNDA
- C212 pad 2: GNDD -> GNDA
- C22 pad 2: GNDD -> GNDA
- C23 pad 2: GNDD -> GNDA
- C24 pad 2: GNDD -> GNDA
- C25 pad 2: GNDD -> GNDA
- C26 pad 2: GNDD -> GNDA
- C27 pad 1: GNDD -> GNDA
- C28 pad 2: GNDD -> GNDA
- C29 pad 2: GNDD -> GNDA
- C3 pad 2: GNDD -> GNDA
- C30 pad 2: GNDD -> GNDA
- C31 pad 1: GNDD -> GNDA
- C32 pad 1: Net-(U19-VI) -> Net-(C20-Pad1)
- C32 pad 2: Net-(C20-Pad2) -> Net-(U19-VI)
- C33 pad 2: GNDD -> GNDA
- C34 pad 2: GNDD -> GNDA
- C36 pad 2: GNDD -> GNDA
- C38 pad 1: GNDD -> GNDA
- C4 pad 2: GNDD -> GNDA
- C40 pad 1: GNDD -> GNDA
- C43 pad 1: Net-(U19-VI) -> Net-(C20-Pad1)
- C43 pad 2: Net-(C20-Pad2) -> Net-(U19-VI)
- C45 pad 1: Net-(U19-VI) -> Net-(C20-Pad1)
- C45 pad 2: Net-(C20-Pad2) -> Net-(U19-VI)
- C47 pad 1: Net-(U19-VI) -> Net-(C20-Pad1)
- C47 pad 2: Net-(C20-Pad2) -> Net-(U19-VI)
- C48 pad 1: GNDD -> GNDA
- C49 pad 2: GNDD -> GNDA
- C5 pad 2: GNDD -> GNDA
- C50 pad 2: GNDD -> GNDA
- C51 pad 2: GNDD -> GNDA
- C52 pad 1: GNDD -> GNDA
- C55 pad 2: GNDD -> GNDA
- C56 pad 1: GNDD -> GNDA
- C59 pad 1: /ADC/+6V -> GNDA
- C59 pad 2: GNDD -> /ADC Range/+12V
- C6 pad 2: GNDD -> GNDA
- C61 pad 1: GNDD -> GNDA
- C62 pad 1: GNDD -> GNDA
- C63 pad 1: GNDD -> GNDA
- C64 pad 1: GNDD -> GNDA
- C65 pad 1: GNDD -> GNDA
- C66 pad 1: GNDD -> GNDA
- C69 pad 2: GNDD -> GNDA
- C7 pad 2: GNDD -> GNDA
- C70 pad 1: GNDD -> GNDA
- C71 pad 2: GNDD -> GNDA
- C72 pad 2: GNDD -> GNDA
- C73 pad 2: GNDD -> GNDA
- C74 pad 2: GNDD -> GNDA
- C75 pad 2: GNDD -> GNDA
- C76 pad 1: GNDD -> GNDA
- C77 pad 2: GNDD -> GNDA
- C78 pad 1: GNDD -> GNDA
- C79 pad 2: GNDD -> GNDA
- C8 pad 2: GNDD -> GNDA
- C80 pad 1: GNDD -> GNDA
- C81 pad 2: GNDD -> GNDA
- C82 pad 1: GNDD -> GNDA
- C83 pad 2: GNDD -> GNDA
- C84 pad 1: GNDD -> GNDA
- C85 pad 2: GNDD -> GNDA
- C86 pad 2: GNDD -> GNDA
- C87 pad 2: GNDD -> GNDA
- C88 pad 1: GNDD -> /ADC/+5V
- C88 pad 2: /ADC/-5V -> GNDA
- C9 pad 1: GNDD -> GNDA
- C91 pad 2: GNDD -> GNDA
- C92 pad 2: GNDD -> GNDA
- C93 pad 1: /ADC/+5V -> /ADC/-5V
- C93 pad 2: GNDD -> GNDA
- C94 pad 2: GNDD -> GNDA
- C95 pad 2: GNDD -> GNDA
- C98 pad 1: GNDD -> GNDA
- C99 pad 2: GNDD -> GNDA
- D1 pad 1: GNDD -> GNDA
- D19 pad 1: GNDD -> GNDA
- D2 pad 1: GNDD -> GNDA
- D3 pad 1: GNDD -> GNDA
- D4 pad 1: GNDD -> GNDA
- D5 pad 2: GNDD -> GNDA
- D6 pad 2: GNDD -> GNDA
- GND_LINK1 pad 1: GNDD -> GNDA
- GND_LINK2 pad 1: GNDD -> GNDA
- GND_LINK2 pad 2: GNDD -> GNDA
- J6 pad 2: GNDD -> GNDA
- J7 pad 2: GNDD -> GNDA
- J8 pad 2: GNDD -> GNDA
- J9 pad 2: GNDD -> GNDA
- M1 pad 1: /ADC/ADC1SCK -> /ADC/ADC2SCK
- M1 pad 10: GNDD -> /DAC/DB0
- M1 pad 2: /ADC/ADC1MISO -> /ADC/ADC2MISO
- M1 pad 25: GNDD -> GNDA
- M1 pad 26: /DAC/DB12 -> /DAC/DB14
- M1 pad 27: /DAC/DB13 -> /DAC/DB15
- M1 pad 28: /DAC/DB14 -> /DAC/DB13
- M1 pad 29: /DAC/DB15 -> /DAC/DB12
- M1 pad 4: /ADC/ADC2SCK -> /ADC/ADC1SCK
- M1 pad 5: /ADC/ADC2MISO -> /ADC/ADC1MISO
- R118 pad 2: GNDD -> GNDA
- R119 pad 2: GNDD -> GNDA
- R27 pad 1: GNDD -> GNDA
- R27 pad 3: GNDD -> GNDA
- R27 pad 5: GNDD -> GNDA
- R27 pad 7: GNDD -> GNDA
- R32 pad 1: GNDD -> GNDA
- R33 pad 1: GNDD -> GNDA
- R33 pad 2: Net-(C20-Pad2) -> Net-(C20-Pad1)
- R43 pad 1: GNDD -> GNDA
- R44 pad 1: GNDD -> GNDA
- R49 pad 1: GNDD -> GNDA
- R50 pad 2: GNDD -> GNDA
- R57 pad 1: GNDD -> GNDA
- R58 pad 1: GNDD -> GNDA
- R59 pad 2: GNDD -> GNDA
- R60 pad 1: GNDD -> GNDA
- R64 pad 1: Net-(C109-Pad2) -> Net-(C113-Pad1)
- R64 pad 2: Net-(C113-Pad1) -> Net-(C109-Pad2)
- R67 pad 1: GNDD -> GNDA
- R68 pad 1: GNDD -> GNDA
- R75 pad 1: GNDD -> GNDA
- R76 pad 1: GNDD -> GNDA
- R8 pad 1: GNDD -> GNDA
- U1 pad 1: GNDD -> GNDA
- U1 pad 10: GNDD -> GNDA
- U1 pad 11: GNDD -> GNDA
- U1 pad 17: GNDD -> GNDA
- U1 pad 2: GNDD -> GNDA
- U1 pad 5: GNDD -> GNDA
- U1 pad 8: GNDD -> GNDA
- U10 pad CN10_20: GNDD -> GNDA
- U10 pad CN10_32: GNDD -> GNDA
- U10 pad CN10_9: GNDD -> GNDA
- U10 pad CN5_7: GNDD -> GNDA
- U10 pad CN6_6: GNDD -> GNDA
- U10 pad CN6_7: GNDD -> GNDA
- U10 pad CN7_19: GNDD -> GNDA
- U10 pad CN7_20: GNDD -> GNDA
- U10 pad CN7_22: GNDD -> GNDA
- U10 pad CN7_8: GNDD -> GNDA
- U12 pad 4: GNDD -> GNDA
- U13 pad 4: GNDD -> GNDA
- U15 pad 7: GNDD -> GNDA
- U16 pad 10: GNDD -> GNDA
- U16 pad 12: GNDD -> GNDA
- U16 pad 13: GNDD -> GNDA
- U16 pad 16: GNDD -> GNDA
- U16 pad 2: GNDD -> GNDA
- U16 pad 3: GNDD -> GNDA
- U16 pad 6: GNDD -> GNDA
- U16 pad 7: GNDD -> GNDA
- U16 pad 8: GNDD -> GNDA
- U16 pad 9: GNDD -> GNDA
- U18 pad 2: GNDD -> GNDA
- U19 pad 1: GNDD -> GNDA
- U2 pad 1: GNDD -> GNDA
- U2 pad 10: GNDD -> GNDA
- U2 pad 11: GNDD -> GNDA
- U2 pad 17: GNDD -> GNDA
- U2 pad 2: GNDD -> GNDA
- U2 pad 5: GNDD -> GNDA
- U2 pad 8: GNDD -> GNDA
- U20 pad 2: GNDD -> GNDA
- U21 pad 1: GNDD -> GNDA
- U22 pad 2: GNDD -> GNDA
- U23 pad 1: GNDD -> GNDA
- U25 pad 13: GNDD -> GNDA
- U25 pad 16: GNDD -> GNDA
- U26 pad 10: GNDD -> GNDA
- U26 pad 12: GNDD -> GNDA
- U26 pad 13: GNDD -> GNDA
- U26 pad 16: GNDD -> GNDA
- U26 pad 2: GNDD -> GNDA
- U26 pad 3: GNDD -> GNDA
- U26 pad 6: GNDD -> GNDA
- U26 pad 7: GNDD -> GNDA
- U26 pad 8: GNDD -> GNDA
- U26 pad 9: GNDD -> GNDA
- U27 pad 13: GNDD -> GNDA
- U27 pad 8: GNDD -> GNDA
- U28 pad 1: GNDD -> GNDA
- U28 pad 3: Net-(U28-VI) -> /ADC/+5V
- U30 pad 12: GNDD -> GNDA
- U30 pad 13: GNDD -> GNDA
- U30 pad 16: GNDD -> GNDA
- U30 pad 2: GNDD -> GNDA
- U30 pad 3: GNDD -> GNDA
- U30 pad 6: GNDD -> GNDA
- U30 pad 9: GNDD -> GNDA
- U31 pad 10: GNDD -> GNDA
- U31 pad 12: GNDD -> GNDA
- U31 pad 13: GNDD -> GNDA
- U31 pad 16: GNDD -> GNDA
- U31 pad 2: GNDD -> GNDA
- U31 pad 3: GNDD -> GNDA
- U31 pad 6: GNDD -> GNDA
- U31 pad 7: GNDD -> GNDA
- U31 pad 8: GNDD -> GNDA
- U31 pad 9: GNDD -> GNDA
- U32 pad 15: GNDD -> GNDA
- U33 pad 10: GNDD -> GNDA
- U33 pad 12: GNDD -> GNDA
- U33 pad 13: GNDD -> GNDA
- U33 pad 16: GNDD -> GNDA
- U33 pad 2: GNDD -> GNDA
- U33 pad 3: GNDD -> GNDA
- U33 pad 6: GNDD -> GNDA
- U33 pad 7: GNDD -> GNDA
- U33 pad 8: GNDD -> GNDA
- U33 pad 9: GNDD -> GNDA
- U35 pad 13: GNDD -> GNDA
- U35 pad 16: GNDD -> GNDA
- U5 pad 4: GNDD -> GNDA
- U6 pad 14: GNDD -> /DAC/DB0
- U6 pad 17: GNDD -> GNDA
- U6 pad 18: GNDD -> GNDA
- U6 pad 24: GNDD -> GNDA
- U7 pad 4: GNDD -> GNDA
Routing:
- net Net-(D9-A): track 0.00 -> 323.7 mm, vias 0 -> 1
- net Net-(D11-A): track 0.00 -> 319.1 mm, vias 0 -> 2
- net Net-(D14-A): track 0.00 -> 317.3 mm, vias 0 -> 1
- net Net-(D8-A): track 0.00 -> 300.4 mm
- net Net-(D10-A): track 0.00 -> 299.7 mm, vias 0 -> 2
- net Net-(D15-A): track 0.00 -> 299.1 mm, vias 0 -> 1
- net /Digital/+3V3: track 0.00 -> 287.7 mm
- net Net-(D13-A): track 0.00 -> 274.5 mm, vias 0 -> 1
- net Net-(U25-A2): track 0.00 -> 257.6 mm, vias 0 -> 3
- net Net-(U32A-A1): track 0.00 -> 234.1 mm, vias 0 -> 4
- net Net-(U25-A1): track 0.00 -> 216.3 mm, vias 0 -> 5
- net /ADC/+5V: track 48.0 -> 260.9 mm, vias 0 -> 3
- net Net-(U32A-ENABLE): track 0.00 -> 211.8 mm, vias 0 -> 2
- net Net-(U32A-A0): track 0.00 -> 211.3 mm, vias 0 -> 3
- net Net-(U25-A0): track 0.00 -> 196.4 mm, vias 0 -> 3
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- added copper zone on In2.Cu, net /+5V_MW
- added copper zone on In2.Cu, net Net-(U18-VI)
- added copper zone on In2.Cu, net Net-(U19-VI)

Commit message: pcb 92%
Parts:
- moved C11 3.02 mm to (106.0, 156.0), turned to 180 degrees
Routing:
- net /Digital/DB1: track 109.7 -> 0.00 mm
- net /Digital/DB2: track 107.9 -> 0.00 mm, vias 1 -> 0
- net /Digital/DB3: track 0.08 -> 87.8 mm, vias 0 -> 2
- net /Digital/DB5: track 0.00 -> 86.3 mm
- net /Digital/DB12: track 69.6 -> 0.00 mm, vias 1 -> 0
- net /Digital/DB6: track 42.7 -> 0.00 mm
- net /Digital/DB4: track 70.7 -> 99.7 mm, vias 0 -> 1
- net Net-(U32A-A0): track 211.3 -> 212.3 mm
- net Net-(U32A-ENABLE): track 211.8 -> 212.8 mm
- net Net-(U32A-A1): track 234.1 -> 234.9 mm

Commit message: pcb update
Parts:
- moved GND_LINK1 13.3 mm to (216.9, 143.6)
Routing:
- net /Digital/DB2: track 0.00 -> 144.2 mm, vias 0 -> 1
- net /Digital/DB1: track 0.00 -> 136.5 mm
- net /Digital/DB12: track 0.00 -> 70.3 mm, vias 0 -> 2
