File: Billeder/DAC_FILTER/DAC_FILTER/DAC_AMP_SCHEMATIC.kicad_sch (KiCad schematic)
At the start: 0 parts

Commit message: STM32 SimpleSample code with PGA and range
Parts:
- added 2Ro: 20, symbol Device:R_US
- added D1, D12, D16, D2: 1N4148, Diode_THT:D_DO-35_SOD27_P7.62mm_Horizontal, symbol Diode:1N4148
- added I1: VDependantISource, symbol JRIX Sources:VDependantISource
- added Q1, Q3: BC547, Package_TO_SOT_THT:TO-92_Inline, symbol Transistor_BJT:BC547
- added Q2, Q4: BC557, Package_TO_SOT_THT:TO-92_Inline, symbol Transistor_BJT:BC557
- added RB (x2), RB1, RB2: 330, symbol Device:R_US
- added RB/2: 165, symbol Device:R_US
- added R_Range, Rd/2: ~, symbol Device:R_US
- added Re (x2), Re1, Re2, Ro, Ro1: 10, symbol Device:R_US
- added Re/2: 5, symbol Device:R_US
- added Rx/2: 26, symbol Device:R_US
- added Z_DUT (x2), Zμ/2, Zπ/2: ~, symbol Device:R
Connections:
- new net: D1.2 (A), Q3.2 (B), RB1.2
- new net: RB/2.2, Rd/2.2, Rx/2.1
- new net: Re1.2, Re2.1, Ro1.1
- new net: Q4.3 (E), Re2.2
- new net: D12.2 (A), Q1.2 (B), RB.2
- new net: D16.1 (K), Q2.2 (B), RB.1
- new net: R_Range.1, Z_DUT.1
- new net: Ro1.2, Z_DUT.2
- new net: I1., Re/2.1, Zπ/2.2
- new net: 2Ro.2, Re/2.2
- new net: D2.1 (K), Q4.2 (B), RB2.1
- new net: Re.1, Re.2, Ro.1
- new net: R_Range.2, Ro.2
- new net: Q2.3 (E), Re.2
- new net: Rx/2.2, Zμ/2.1, Zπ/2.1
- new net: Q3.3 (E), Re1.1
- new net: Q1.3 (E), Re.1
- new net +5V: Q1.1 (C), Q3.1 (C), RB.1, RB1.1
- new net -5V: Q2.1 (C), Q4.1 (C), RB.2, RB2.2
- new net DAC+: D12.1 (K), D16.2 (A)
- new net DAC-: D1.1 (K), D2.2 (A)
- new net GND: I1., RB/2.1, Z_DUT.2, Zμ/2.2
- new net Vi: Rd/2.1
- new net Vo: 2Ro.1, Z_DUT.1
Other:
- note added: "2gm·Vπ = i2·2gm·(Zπ/2) = i2·gm·Zπ"
- note added: "i1"
- note added: "i2"
- note added: "i3"
