File: Billeder/DAC_FILTER/DAC_FILTER/DAC_PZ.kicad_sch (KiCad schematic)
At the start: 6 parts

Commit message: DAC Power Stability
Parts:
- added Rx/2: 51, symbol Device:R_US
Connections:
- net at Z_π/2.1: now also Rx/2.2; no longer Rd/2.2
- new net: Rd/2.2, Rx/2.1
Other:
- moved on the sheet: Rd/2, Z_π/2
Changed lines of the file:
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@@
+	(wire
+		(pts
+			(xy 110.49 85.09) (xy 114.3 85.09)
+		)
+		(stroke
+			(width 0)
+			(type default)
+		)
+	)
 	(wire
 		(pts
@@
 	(wire
 		(pts
+			(xy 121.92 85.09) (xy 127 85.09)
+		)
+		(stroke
+			(width 0)
+			(type default)
+		)
+	)
+	(wire
+		(pts
 			(xy 157.48 85.09) (xy 168.91 85.09)
 		)
@@
 	(wire
 		(pts
-			(xy 129.54 85.09) (xy 142.24 85.09)
+			(xy 134.62 85.09) (xy 142.24 85.09)
 		)
 		(stroke
@@
 	(wire
 		(pts
-			(xy 102.87 85.09) (xy 105.41 85.09)
-		)
-		(stroke
-			(width 0)
-			(type default)
-		)
-	)
-	(wire
-		(pts
-			(xy 113.03 85.09) (xy 121.92 85.09)
+			(xy 99.06 85.09) (xy 102.87 85.09)
 		)
 		(stroke
@@
 	(text "Z_π = 0\nat High Frequencies"
 		(exclude_from_sim no)
-		(at 120.904 90.17 0)
+		(at 124.46 90.17 0)
 		(effects
 			(font
@@
 	(global_label "Vi"
 		(shape input)
-		(at 102.87 85.09 180)
+		(at 99.06 85.09 180)
 		(fields_autoplaced yes)
 		(effects
@@
 		)
 		(property "Intersheetrefs" "${INTERSHEET_REFS}"
-			(at 98.1914 85.09 0)
+			(at 94.3814 85.09 0)
 			(effects
 				(font
@@
 	(symbol
 		(lib_id "Device:R")
-		(at 125.73 85.09 90)
+		(at 130.81 85.09 90)
 		(unit 1)
 		(exclude_from_sim no)
@@
 		(fields_autoplaced yes)
 		(property "Reference" "Z_π/2"
-			(at 125.73 80.01 90)
+			(at 130.81 80.01 90)
 			(effects
 				(font
@@
 		)
 		(property "Value" "~"
-			(at 125.73 82.55 90)
-			(effects
-				(font
-					(size 1.27 1.27)
-				)
-			)
-		)
-		(property "Footprint" ""
-			(at 125.73 86.868 90)
-			(effects
-				(font
-					(size 1.27 1.27)
-				)
-				(hide yes)
-			)
-		)
-		(property "Datasheet" "~"
-			(at 125.73 85.09 0)
+			(at 130.81 82.55 90)
+			(effects
+				(font
+					(size 1.27 1.27)
+				)
+			)
+		)
+		(property "Footprint" ""
+			(at 130.81 86.868 90)
+			(effects
+				(font
+					(size 1.27 1.27)
+				)
+				(hide yes)
+			)
+		)
+		(property "Datasheet" "~"
+			(at 130.81 85.09 0)
 			(effects
 				(font
@@
 		)
 		(property "Description" "Resistor"
-			(at 125.73 85.09 0)
+			(at 130.81 85.09 0)
 			(effects
 				(font
@@
 	(symbol
 		(lib_id "Device:R_US")
-		(at 109.22 85.09 90)
+		(at 118.11 85.09 90)
+		(unit 1)
+		(exclude_from_sim no)
+		(in_bom yes)
+		(on_board yes)
+		(dnp no)
+		(fields_autoplaced yes)
+		(property "Reference" "Rx/2"
+			(at 118.11 78.74 90)
+			(effects
+				(font
+					(size 1.27 1.27)
+				)
+			)
+		)
+		(property "Value" "51"
+			(at 118.11 81.28 90)
+			(effects
+				(font
+					(size 1.27 1.27)
+				)
+			)
+		)
+		(property "Footprint" ""
+			(at 118.364 84.074 90)
+			(effects
+				(font
+					(size 1.27 1.27)
+				)
+				(hide yes)
+			)
+		)
+		(property "Datasheet" "~"
+			(at 118.11 85.09 0)
+			(effects
+				(font
+					(size 1.27 1.27)
+				)
+				(hide yes)
+			)
+		)
+		(property "Description" "Resistor, US symbol"
+			(at 118.11 85.09 0)
+			(effects
+				(font
+					(size 1.27 1.27)
+				)
+				(hide yes)
+			)
+		)
+		(pin "1"
+		)
+		(pin "2"
+		)
+		(instances
+			(project "DAC_FILTER"
+				(path "/5ea4bdd8-845d-49bd-9427-a30bfd0e620f/b81d1699-6837-4e16-b045-af8fdd78bc85"
+					(reference "Rx/2")
+					(unit 1)
+				)
+			)
+		)
+	)
+	(symbol
+		(lib_id "Device:R_US")
+		(at 106.68 85.09 90)
 		(unit 1)
 		(exclude_from_sim no)
@@
 		(fields_autoplaced yes)
 		(property "Reference" "Rd/2"
-			(at 109.22 78.74 90)
+			(at 106.68 78.74 90)
 			(effects
 				(font
@@
 		)
 		(property "Value" "2"
-			(at 109.22 81.28 90)
-			(effects
-				(font
-					(size 1.27 1.27)
-				)
-			)
-		)
-		(property "Footprint" ""
-			(at 109.474 84.074 90)
-			(effects
-				(font
-					(size 1.27 1.27)
-				)
-				(hide yes)
-			)
-		)
-		(property "Datasheet" "~"
-			(at 109.22 85.09 0)
+			(at 106.68 81.28 90)
+			(effects
+				(font
+					(size 1.27 1.27)
+				)
+			)
+		)
+		(property "Footprint" ""
+			(at 106.934 84.074 90)
+			(effects
+				(font
+					(size 1.27 1.27)
+				)
+				(hide yes)
+			)
+		)
+		(property "Datasheet" "~"
+			(at 106.68 85.09 0)
 			(effects
 				(font
@@
 		)
 		(property "Description" "Resistor, US symbol"
-			(at 109.22 85.09 0)
-			(effects
-				(font
+			(at 106.68 85.09 0)
+			(effects
+				(font
