File: Billeder/DAC_FILTER/DAC_FILTER/DAC_SIM_MODEL.kicad_sch (KiCad schematic)
At the start: 14 parts

Commit message: DAC Power Stability
Parts:
- Rx/2: value 256 -> 51
- Rπ/2: value 1024 -> 256
Changed lines of the file:
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@@
 			)
 		)
-		(property "Value" "1024"
+		(property "Value" "256"
 			(at 158.75 77.4699 0)
 			(effects
@@
 			)
 		)
-		(property "Value" "256"
+		(property "Value" "51"
 			(at 133.35 63.5 90)
 			(effects
